Commit message: 210726 settings upload

File: op3_gym/urdf_simple/robotis_op3.gazebo.xacro (robot description, xacro)
@@ -11,5 +11,5 @@
     <mu2>0.2</mu2>
     <material>Gazebo/White</material>
-    <selfCollide>true</selfCollide>
+    <selfCollide>false</selfCollide>
   </gazebo>
   <!-- left leg links -->
@@ -18,5 +18,5 @@
     <mu2>0.2</mu2>
     <material>Gazebo/White</material>
-    <selfCollide>true</selfCollide>
+    <selfCollide>false</selfCollide>
   </gazebo>
   <gazebo reference="l_hip_roll_link">
@@ -24,5 +24,5 @@
     <mu2>0.2</mu2>
     <material>Gazebo/White</material>
-    <selfCollide>true</selfCollide>
+    <selfCollide>false</selfCollide>
   </gazebo>
   <gazebo reference="l_hip_pitch_link">
@@ -30,5 +30,5 @@
     <mu2>0.2</mu2>
     <material>Gazebo/White</material>
-    <selfCollide>true</selfCollide>
+    <selfCollide>false</selfCollide>
   </gazebo>
   <gazebo reference="l_knee_link">
@@ -36,5 +36,5 @@
     <mu2>0.2</mu2>
     <material>Gazebo/White</material>
-    <selfCollide>true</selfCollide>
+    <selfCollide>false</selfCollide>
   </gazebo>
   <gazebo reference="l_ank_pitch_link">
@@ -42,5 +42,5 @@
     <mu2>0.2</mu2>
     <material>Gazebo/White</material>
-    <selfCollide>true</selfCollide>
+    <selfCollide>false</selfCollide>
   </gazebo>
   <gazebo reference="l_ank_roll_link">
@@ -59,5 +59,5 @@
     <mu2>0.2</mu2>
     <material>Gazebo/White</material>
-    <selfCollide>true</selfCollide>
+    <selfCollide>false</selfCollide>
   </gazebo>
   <gazebo reference="r_hip_roll_link">
@@ -65,5 +65,5 @@
     <mu2>0.2</mu2>
     <material>Gazebo/White</material>
-    <selfCollide>true</selfCollide>
+    <selfCollide>false</selfCollide>
   </gazebo>
   <gazebo reference="r_hip_pitch_link">
@@ -71,5 +71,5 @@
     <mu2>0.2</mu2>
     <material>Gazebo/White</material>
-    <selfCollide>true</selfCollide>
+    <selfCollide>false</selfCollide>
   </gazebo>
   <gazebo reference="r_knee_link">
@@ -77,5 +77,5 @@
     <mu2>0.2</mu2>
     <material>Gazebo/White</material>
-    <selfCollide>true</selfCollide>
+    <selfCollide>false</selfCollide>
   </gazebo>
   <gazebo reference="r_ank_pitch_link">
@@ -83,5 +83,5 @@
     <mu2>0.2</mu2>
     <material>Gazebo/White</material>
-    <selfCollide>true</selfCollide>
+    <selfCollide>false</selfCollide>
   </gazebo>
   <gazebo reference="r_ank_roll_link">
@@ -100,5 +100,5 @@
     <mu2>0.2</mu2>
     <material>Gazebo/White</material>
-    <selfCollide>true</selfCollide>
+    <selfCollide>false</selfCollide>
   </gazebo>
   <gazebo reference="r_sho_roll_link">
@@ -106,5 +106,5 @@
     <mu2>0.2</mu2>
     <material>Gazebo/White</material>
-    <selfCollide>true</selfCollide>
+    <selfCollide>false</selfCollide>
   </gazebo>
   <gazebo reference="r_el_link">
@@ -112,5 +112,5 @@
     <mu2>0.2</mu2>
     <material>Gazebo/White</material>
-    <selfCollide>true</selfCollide>
+    <selfCollide>false</selfCollide>
   </gazebo>
   <gazebo reference="l_sho_pitch_link">
@@ -118,5 +118,5 @@
     <mu2>0.2</mu2>
     <material>Gazebo/White</material>
-    <selfCollide>true</selfCollide>
+    <selfCollide>false</selfCollide>
   </gazebo>
   <gazebo reference="l_sho_roll_link">
@@ -124,5 +124,5 @@
     <mu2>0.2</mu2>
     <material>Gazebo/White</material>
-    <selfCollide>true</selfCollide>
+    <selfCollide>false</selfCollide>
   </gazebo>
   <gazebo reference="l_el_link">
@@ -130,5 +130,5 @@
     <mu2>0.2</mu2>
     <material>Gazebo/White</material>
-    <selfCollide>true</selfCollide>
+    <selfCollide>false</selfCollide>
   </gazebo>
   <gazebo reference="head_pan_link">
@@ -136,5 +136,5 @@
     <mu2>0.2</mu2>
     <material>Gazebo/White</material>
-    <selfCollide>true</selfCollide>
+    <selfCollide>false</selfCollide>
   </gazebo>
   <gazebo reference="head_tilt_link">
@@ -142,5 +142,5 @@
     <mu2>0.2</mu2>
     <material>Gazebo/White</material>
-    <selfCollide>true</selfCollide>
+    <selfCollide>false</selfCollide>
   </gazebo>
 <!--
@@ -265,5 +265,5 @@
     <sensor name="imu_sensor" type="imu">
       <always_on>true</always_on>
-      <update_rate>400</update_rate>
+      <update_rate>100</update_rate>
       <visualize>true</visualize>
       <topic>__default_topic__</topic>
@@ -271,5 +271,5 @@
         <topicName>robotis_op3/imu</topicName>
         <bodyName>body_link</bodyName>
-        <updateRateHZ>0</updateRateHZ>
+        <updateRateHZ>10.0</updateRateHZ>
         <gaussianNoise>0.0</gaussianNoise>
         <xyzOffset>0 0 0</xyzOffset>

File: op3_gym/urdf_simple/robotis_op3.structure.head.xacro (robot description, xacro)
@@ -12,6 +12,6 @@
     <origin xyz="-0.001 0.0 0.1365" rpy="0 0 0" />
     <axis xyz="0 0 1" />
-    <limit effort="1.5" velocity="100" lower="${-pi*0.9}" upper="${pi*0.9}" />
-    <dynamics damping="0.1" friction="0.0" />
+    <limit effort="1.51" velocity="100" lower="${-pi*0.9}" upper="${pi*0.9}" />
+    <dynamics damping="0.01" friction="0.0" />
   </joint>
   <xacro:insert_transmission name="head_pan" />
@@ -21,7 +21,7 @@
       <xacro:insert_mesh_head_pan_link />
     </visual>
-    <collision>
+    <!-- <collision>
       <xacro:insert_mesh_head_pan_link />
-    </collision>
+    </collision> -->
     <inertial>
       <xacro:insert_inertia_head_pan_link />
@@ -34,6 +34,6 @@
     <origin xyz="0.010 0.019 0.0285" rpy="0 0 0" />
     <axis xyz="0 -1 0" />
-    <limit effort="1.5" velocity="100" lower="${-pi*0.9}" upper="${pi*0.9}" />
-    <dynamics damping="0.1" friction="0.0" />
+    <limit effort="1.51" velocity="100" lower="${-pi*0.9}" upper="${pi*0.9}" />
+    <dynamics damping="0.01" friction="0.0" />
   </joint>
   <xacro:insert_transmission name="head_tilt" />
@@ -43,7 +43,7 @@
       <xacro:insert_mesh_head_tilt_link />
     </visual>
-    <collision>
+    <!-- <collision>
       <xacro:insert_mesh_head_tilt_link />
-    </collision>
+    </collision> -->
     <inertial>
       <xacro:insert_inertia_head_tilt_link />
@@ -51,20 +51,20 @@
   </link>
   <!-- camera joint -->
-  <!--
-    <joint name="cam" type="fixed">
-      <origin xyz="0.01425 -0.019 0.04975" rpy="${-pi*0.5} 0 ${-pi*0.5}"/>
-      <parent link="head_tilt_link"/>
-      <child link="cam_link"/>
-    </joint>
-    <joint name="cam_gazebo" type="fixed">
-      <origin xyz="0.01425 -0.019 0.04975" rpy="0 0 0"/>
-      <parent link="head_tilt_link"/>
-      <child link="cam_gazebo_link"/>
-    </joint>
-    <link name="cam_link">
-    </link>
-    <link name="cam_gazebo_link">
-    </link>
-  -->
+  <!-- <joint name="cam" type="fixed">
+    <origin xyz="0.01425 -0.019 0.04975" rpy="${-pi*0.5} 0 ${-pi*0.5}"/>
+    <parent link="head_tilt_link"/>
+    <child link="cam_link"/>
+  </joint> -->
+  <!-- <joint name="cam_gazebo" type="fixed">
+    <origin xyz="0.01425 -0.019 0.04975" rpy="0 0 0"/>
+    <parent link="head_tilt_link"/>
+    <child link="cam_gazebo_link"/>
+  </joint> -->
+  <!-- camera link -->
+  <!-- <link name="cam_link">
+  </link> -->
+  <!-- camera link -->
+  <!-- <link name="cam_gazebo_link">
+  </link> -->
   </xacro:macro>
 </robot>

File: op3_gym/urdf_simple/robotis_op3.structure.larm.xacro (robot description, xacro)
@@ -12,6 +12,6 @@
     <origin xyz="-0.001 0.06 0.111" rpy="0 0 0" />
     <axis xyz="0 1 0" />
-    <limit effort="1.5" velocity="100" lower="${-pi*0.9}" upper="${pi*0.9}" />
-    <dynamics damping="0.1" friction="0.01" />
+    <limit effort="1.51" velocity="100" lower="${-pi*0.9}" upper="${pi*0.9}" />
+    <dynamics damping="0.01" friction="0.0" />
   </joint>
   <xacro:insert_transmission name="l_sho_pitch" />
@@ -21,7 +21,7 @@
       <xacro:insert_mesh_l_sho_pitch_link />
     </visual>
-    <collision>
+    <!-- <collision>
       <xacro:insert_mesh_l_sho_pitch_link />
-    </collision>
+    </collision> -->
     <inertial>
       <xacro:insert_inertia_l_sho_pitch_link />
@@ -34,6 +34,6 @@
     <origin xyz="0.019 0.0285 -0.010" rpy="0 0 0" />
     <axis xyz="-1 0 0" />
-    <limit effort="1.5" velocity="100" lower="${-pi*0.9}" upper="${pi*0.9}" />
-    <dynamics damping="0.1" friction="0.01" />
+    <limit effort="1.51" velocity="100" lower="${-pi*0.9}" upper="${pi*0.9}" />
+    <dynamics damping="0.01" friction="0.0" />
   </joint>
   <xacro:insert_transmission name="l_sho_roll" />
@@ -43,7 +43,7 @@
       <xacro:insert_mesh_l_sho_roll_link />
     </visual>
-    <collision>
+    <!-- <collision>
       <xacro:insert_mesh_l_sho_roll_link />
-    </collision>
+    </collision> -->
     <inertial>
       <xacro:insert_inertia_l_sho_roll_link />
@@ -56,6 +56,6 @@
     <origin xyz="0.0 0.0904 -0.0001" rpy="0 0 0" />
     <axis xyz="1 0 0" />
-    <limit effort="1.5" velocity="100" lower="${-pi*0.9}" upper="${pi*0.9}" />
-    <dynamics damping="0.1" friction="0.01" />
+    <limit effort="1.51" velocity="100" lower="${-pi*0.9}" upper="${pi*0.9}" />
+    <dynamics damping="0.01" friction="0.0" />
   </joint>
   <xacro:insert_transmission name="l_el" />
@@ -65,7 +65,7 @@
       <xacro:insert_mesh_l_el_link />
     </visual>
-    <collision>
+    <!-- <collision>
       <xacro:insert_mesh_l_el_link />
-    </collision>
+    </collision> -->
     <inertial>
       <xacro:insert_inertia_l_el_link />

File: op3_gym/urdf_simple/robotis_op3.structure.lleg.xacro (robot description, xacro)
@@ -12,6 +12,6 @@
     <origin xyz="0.0 0.035 0.0" rpy="0 0 0" />
     <axis xyz="0 0 -1" />
-    <limit effort="1.5" velocity="100" lower="${-pi*0.9}" upper="${pi*0.9}" />
-    <dynamics damping="0.1" friction="0.0" />
+    <limit effort="1.51" velocity="100" lower="${-pi*0.9}" upper="${pi*0.9}" />
+    <dynamics damping="0.01" friction="0.0" />
   </joint>
   <xacro:insert_transmission name="l_hip_yaw" />
@@ -21,7 +21,7 @@
       <xacro:insert_mesh_l_hip_yaw_link />
     </visual>
-    <collision>
+    <!-- <collision>
       <xacro:insert_mesh_l_hip_yaw_link />
-    </collision>
+    </collision> -->
     <inertial>
       <xacro:insert_inertia_l_hip_yaw_link />
@@ -34,6 +34,6 @@
     <origin xyz="-0.024 0.0 -0.0285" rpy="0 0 0" />
     <axis xyz="-1 0 0" />
-    <limit effort="1.5" velocity="100" lower="${-pi*0.9}" upper="${pi*0.9}" />
-    <dynamics damping="0.1" friction="0.0" />
+    <limit effort="1.51" velocity="100" lower="${-pi*0.9}" upper="${pi*0.9}" />
+    <dynamics damping="0.01" friction="0.0" />
   </joint>
   <xacro:insert_transmission name="l_hip_roll" />
@@ -43,7 +43,7 @@
       <xacro:insert_mesh_l_hip_roll_link />
     </visual>
-    <collision>
+    <!-- <collision>
       <xacro:insert_mesh_l_hip_roll_link />
-    </collision>
+    </collision> -->
     <inertial>
       <xacro:insert_inertia_l_hip_roll_link />
@@ -56,6 +56,6 @@
     <origin xyz="0.0241 0.019 0.0" rpy="0 0 0" />
     <axis xyz="0 1 0" />
-    <limit effort="1.5" velocity="100" lower="${-pi*0.9}" upper="${pi*0.9}" />
-    <dynamics damping="0.1" friction="0.0" />
+    <limit effort="1.51" velocity="100" lower="${-pi*0.9}" upper="${pi*0.9}" />
+    <dynamics damping="0.01" friction="0.0" />
   </joint>
   <xacro:insert_transmission name="l_hip_pitch" />
@@ -66,5 +66,9 @@
     </visual>
     <collision>
-      <xacro:insert_mesh_l_hip_pitch_link />
+      <!-- <xacro:insert_mesh_l_hip_pitch_link /> -->
+      <origin xyz="0.03 -0.05 -0.04" rpy="0.0 0.0 0.0"/>
+      <geometry>
+        <box size="0.03 0.03 0.13"/>
+      </geometry>
     </collision>
     <inertial>
@@ -78,6 +82,6 @@
     <origin xyz="0.0 0.0 -0.11015" rpy="0 0 0" />
     <axis xyz="0 1 0" />
-    <limit effort="1.5" velocity="100" lower="${-pi*0.9}" upper="${pi*0.9}" />
-    <dynamics damping="0.1" friction="0.0" />
+    <limit effort="1.51" velocity="100" lower="${-pi*0.9}" upper="${pi*0.9}" />
+    <dynamics damping="0.01" friction="0.0" />
   </joint>
   <xacro:insert_transmission name="l_knee" />
@@ -88,5 +92,9 @@
     </visual>
     <collision>
-      <xacro:insert_mesh_l_knee_link />
+      <!-- <xacro:insert_mesh_l_knee_link /> -->
+      <origin xyz="0.03 -0.05 -0.05" rpy="0.0 0.0 0.0"/>
+      <geometry>
+        <box size="0.03 0.03 0.1"/>
+      </geometry>
     </collision>
     <inertial>
@@ -100,6 +108,6 @@
     <origin xyz="0 0 -0.110" rpy="0 0 0" />
     <axis xyz="0 -1 0" />
-    <limit effort="1.5" velocity="100" lower="${-pi*0.9}" upper="${pi*0.9}" />
-    <dynamics damping="0.1" friction="0.0" />
+    <limit effort="1.51" velocity="100" lower="${-pi*0.9}" upper="${pi*0.9}" />
+    <dynamics damping="0.01" friction="0.0" />
   </joint>
   <xacro:insert_transmission name="l_ank_pitch" />
@@ -109,7 +117,7 @@
       <xacro:insert_mesh_l_ank_pitch_link />
     </visual>
-    <collision>
+    <!-- <collision>
       <xacro:insert_mesh_l_ank_pitch_link />
-    </collision>
+    </collision> -->
     <inertial>
       <xacro:insert_inertia_l_ank_pitch_link />
@@ -122,6 +130,6 @@
     <origin xyz="-0.0241 -0.019 0" rpy="0 0 0" />
     <axis xyz="1 0 0" />
-    <limit effort="1.5" velocity="100" lower="${-pi*0.9}" upper="${pi*0.9}" />
-    <dynamics damping="0.1" friction="0.0" />
+    <limit effort="1.51" velocity="100" lower="${-pi*0.9}" upper="${pi*0.9}" />
+    <dynamics damping="0.01" friction="0.0" />
   </joint>
   <xacro:insert_transmission name="l_ank_roll" />
@@ -132,5 +140,9 @@
     </visual>
     <collision>
-      <xacro:insert_mesh_l_ank_roll_link />
+      <!-- <xacro:insert_mesh_l_ank_roll_link /> -->
+      <origin xyz="0 0.03 -0.03" rpy="0 0 0" />
+      <geometry>
+        <box size="0.145 0.09 0.01" />
+      </geometry>
     </collision>
     <inertial>

File: op3_gym/urdf_simple/robotis_op3.structure.rarm.xacro (robot description, xacro)
@@ -12,6 +12,6 @@
     <origin xyz="-0.001 -0.06 0.111" rpy="0 0 0" />
     <axis xyz="0 -1 0" />
-    <limit effort="1.5" velocity="100" lower="${-pi*0.9}" upper="${pi*0.9}" />
-    <dynamics damping="0.1" friction="0.0" />
+    <limit effort="1.51" velocity="100" lower="${-pi*0.9}" upper="${pi*0.9}" />
+    <dynamics damping="0.01" friction="0.0" />
   </joint>
   <xacro:insert_transmission name="r_sho_pitch" />
@@ -21,7 +21,7 @@
       <xacro:insert_mesh_r_sho_pitch_link />
     </visual>
-    <collision>
+    <!-- <collision>
       <xacro:insert_mesh_r_sho_pitch_link />
-    </collision>
+    </collision> -->
     <inertial>
       <xacro:insert_inertia_r_sho_pitch_link />
@@ -34,6 +34,6 @@
     <origin xyz="0.019 -0.0285 -0.010" rpy="0 0 0" />
     <axis xyz="-1 0 0" />
-    <limit effort="1.5" velocity="100" lower="${-pi*0.9}" upper="${pi*0.9}" />
-    <dynamics damping="0.1" friction="0.0" />
+    <limit effort="1.51" velocity="100" lower="${-pi*0.9}" upper="${pi*0.9}" />
+    <dynamics damping="0.01" friction="0.0" />
   </joint>
   <xacro:insert_transmission name="r_sho_roll" />
@@ -43,7 +43,7 @@
       <xacro:insert_mesh_r_sho_roll_link />
     </visual>
-    <collision>
+    <!-- <collision>
       <xacro:insert_mesh_r_sho_roll_link />
-    </collision>
+    </collision> -->
     <inertial>
       <xacro:insert_inertia_r_sho_roll_link />
@@ -56,6 +56,6 @@
     <origin xyz="0.0 -0.0904 -0.0001" rpy="0 0 0" />
     <axis xyz="1 0 0" />
-    <limit effort="1.5" velocity="100" lower="${-pi*0.9}" upper="${pi*0.9}" />
-    <dynamics damping="0.1" friction="0.0" />
+    <limit effort="1.51" velocity="100" lower="${-pi*0.9}" upper="${pi*0.9}" />
+    <dynamics damping="0.01" friction="0.0" />
   </joint>
   <xacro:insert_transmission name="r_el" />
@@ -65,7 +65,7 @@
       <xacro:insert_mesh_r_el_link />
     </visual>
-    <collision>
+    <!-- <collision>
       <xacro:insert_mesh_r_el_link />
-    </collision>
+    </collision> -->
     <inertial>
       <xacro:insert_inertia_r_el_link />

File: op3_gym/urdf_simple/robotis_op3.structure.rleg.xacro (robot description, xacro)
@@ -12,6 +12,6 @@
     <origin xyz="0.0 -0.035 0.0" rpy="0 0 0" />
     <axis xyz="0 0 -1" />
-    <limit effort="1.5" velocity="100" lower="${-pi*0.9}" upper="${pi*0.9}" />
-    <dynamics damping="0.1" friction="0.0" />
+    <limit effort="1.51" velocity="100" lower="${-pi*0.9}" upper="${pi*0.9}" />
+    <dynamics damping="0.01" friction="0.0" />
   </joint>
   <xacro:insert_transmission name="r_hip_yaw" />
@@ -21,7 +21,7 @@
       <xacro:insert_mesh_r_hip_yaw_link />
     </visual>
-    <collision>
+    <!-- <collision>
       <xacro:insert_mesh_r_hip_yaw_link />
-    </collision>
+    </collision> -->
     <inertial>
       <xacro:insert_inertia_r_hip_yaw_link />
@@ -34,6 +34,6 @@
     <origin xyz="-0.024 0.0 -0.0285" rpy="0 0 0" />
     <axis xyz="-1 0 0" />
-    <limit effort="1.5" velocity="100" lower="${-pi*0.9}" upper="${pi*0.9}" />
-    <dynamics damping="0.1" friction="0.0" />
+    <limit effort="1.51" velocity="100" lower="${-pi*0.9}" upper="${pi*0.9}" />
+    <dynamics damping="0.01" friction="0.0" />
   </joint>
   <xacro:insert_transmission name="r_hip_roll" />
@@ -43,7 +43,7 @@
       <xacro:insert_mesh_r_hip_roll_link />
     </visual>
-    <collision>
+    <!-- <collision>
       <xacro:insert_mesh_r_hip_roll_link />
-    </collision>
+    </collision> -->
     <inertial>
       <xacro:insert_inertia_r_hip_roll_link />
@@ -56,6 +56,6 @@
     <origin xyz="0.0241 -0.019 0.0" rpy="0 0 0" />
     <axis xyz="0 -1 0" />
-    <limit effort="1.5" velocity="100" lower="${-pi*0.9}" upper="${pi*0.9}" />
-    <dynamics damping="0.1" friction="0.0" />
+    <limit effort="1.51" velocity="100" lower="${-pi*0.9}" upper="${pi*0.9}" />
+    <dynamics damping="0.01" friction="0.0" />
   </joint>
   <xacro:insert_transmission name="r_hip_pitch" />
@@ -66,5 +66,9 @@
     </visual>
     <collision>
-      <xacro:insert_mesh_r_hip_pitch_link />
+      <!-- <xacro:insert_mesh_r_hip_pitch_link /> -->
+      <origin xyz="0.03 0.0 -0.04" rpy="0.0 0.0 0.0"/>
+      <geometry>
+        <box size="0.03 0.03 0.13"/>
+      </geometry>
     </collision>
     <inertial>
@@ -78,6 +82,6 @@
     <origin xyz="0.0 0.0 -0.11015" rpy="0 0 0" />
     <axis xyz="0 -1 0" />
-    <limit effort="1.5" velocity="100" lower="${-pi*0.9}" upper="${pi*0.9}" />
-    <dynamics damping="0.1" friction="0.0" />
+    <limit effort="1.51" velocity="100" lower="${-pi*0.9}" upper="${pi*0.9}" />
+    <dynamics damping="0.01" friction="0.0" />
   </joint>
   <xacro:insert_transmission name="r_knee" />
@@ -88,5 +92,9 @@
     </visual>
     <collision>
-      <xacro:insert_mesh_r_knee_link />
+      <!-- <xacro:insert_mesh_r_knee_link /> -->
+      <origin xyz="0.03 0.0 -0.05" rpy="0.0 0.0 0.0"/>
+      <geometry>
+        <box size="0.03 0.03 0.1"/>
+      </geometry>
     </collision>
     <inertial>
@@ -100,6 +108,6 @@
     <origin xyz="0 0 -0.110" rpy="0 0 0" />
     <axis xyz="0 1 0" />
-    <limit effort="1.5" velocity="100" lower="${-pi*0.9}" upper="${pi*0.9}" />
-    <dynamics damping="0.1" friction="0.0" />
+    <limit effort="1.51" velocity="100" lower="${-pi*0.9}" upper="${pi*0.9}" />
+    <dynamics damping="0.01" friction="0.0" />
   </joint>
   <xacro:insert_transmission name="r_ank_pitch" />
@@ -109,7 +117,7 @@
       <xacro:insert_mesh_r_ank_pitch_link />
     </visual>
-    <collision>
+    <!-- <collision>
       <xacro:insert_mesh_r_ank_pitch_link />
-    </collision>
+    </collision> -->
     <inertial>
       <xacro:insert_inertia_r_ank_pitch_link />
@@ -122,6 +130,6 @@
     <origin xyz="-0.0241 0.019 0" rpy="0 0 0" />
     <axis xyz="1 0 0" />
-    <limit effort="1.5" velocity="100" lower="${-pi*0.9}" upper="${pi*0.9}" />
-    <dynamics damping="0.1" friction="0.0" />
+    <limit effort="1.51" velocity="100" lower="${-pi*0.9}" upper="${pi*0.9}" />
+    <dynamics damping="0.01" friction="0.0" />
   </joint>
   <xacro:insert_transmission name="r_ank_roll" />
@@ -132,5 +140,9 @@
     </visual>
     <collision>
-      <xacro:insert_mesh_r_ank_roll_link />
+      <!-- <xacro:insert_mesh_r_ank_roll_link /> -->
+      <origin xyz="0 0 -0.03" rpy="0 0 0" />
+      <geometry>
+        <box size="0.145 0.09 0.01" />
+      </geometry>
     </collision>
     <inertial>
