Commit message: fix urdf_simple

File: op3_gym/urdf_simple/robotis_op3.structure.head.xacro (robot description, xacro)
@@ -13,5 +13,5 @@
     <axis xyz="0 0 1" />
     <limit effort="1.51" velocity="100" lower="${-pi*0.9}" upper="${pi*0.9}" />
-    <dynamics damping="0.01" friction="0.0" />
+    <dynamics damping="0.1" friction="0.0" />
   </joint>
   <xacro:insert_transmission name="head_pan" />
@@ -35,5 +35,5 @@
     <axis xyz="0 -1 0" />
     <limit effort="1.51" velocity="100" lower="${-pi*0.9}" upper="${pi*0.9}" />
-    <dynamics damping="0.01" friction="0.0" />
+    <dynamics damping="0.1" friction="0.0" />
   </joint>
   <xacro:insert_transmission name="head_tilt" />

File: op3_gym/urdf_simple/robotis_op3.structure.larm.xacro (robot description, xacro)
@@ -13,5 +13,5 @@
     <axis xyz="0 1 0" />
     <limit effort="1.51" velocity="100" lower="${-pi*0.9}" upper="${pi*0.9}" />
-    <dynamics damping="0.01" friction="0.0" />
+    <dynamics damping="0.1" friction="0.0" />
   </joint>
   <xacro:insert_transmission name="l_sho_pitch" />
@@ -35,5 +35,5 @@
     <axis xyz="-1 0 0" />
     <limit effort="1.51" velocity="100" lower="${-pi*0.9}" upper="${pi*0.9}" />
-    <dynamics damping="0.01" friction="0.0" />
+    <dynamics damping="0.1" friction="0.0" />
   </joint>
   <xacro:insert_transmission name="l_sho_roll" />
@@ -57,5 +57,5 @@
     <axis xyz="1 0 0" />
     <limit effort="1.51" velocity="100" lower="${-pi*0.9}" upper="${pi*0.9}" />
-    <dynamics damping="0.01" friction="0.0" />
+    <dynamics damping="0.1" friction="0.0" />
   </joint>
   <xacro:insert_transmission name="l_el" />

File: op3_gym/urdf_simple/robotis_op3.structure.lleg.xacro (robot description, xacro)
@@ -13,5 +13,5 @@
     <axis xyz="0 0 -1" />
     <limit effort="1.51" velocity="100" lower="${-pi*0.9}" upper="${pi*0.9}" />
-    <dynamics damping="0.01" friction="0.0" />
+    <dynamics damping="0.1" friction="0.0" />
   </joint>
   <xacro:insert_transmission name="l_hip_yaw" />
@@ -35,5 +35,5 @@
     <axis xyz="-1 0 0" />
     <limit effort="1.51" velocity="100" lower="${-pi*0.9}" upper="${pi*0.9}" />
-    <dynamics damping="0.01" friction="0.0" />
+    <dynamics damping="0.1" friction="0.0" />
   </joint>
   <xacro:insert_transmission name="l_hip_roll" />
@@ -57,5 +57,5 @@
     <axis xyz="0 1 0" />
     <limit effort="1.51" velocity="100" lower="${-pi*0.9}" upper="${pi*0.9}" />
-    <dynamics damping="0.01" friction="0.0" />
+    <dynamics damping="0.1" friction="0.0" />
   </joint>
   <xacro:insert_transmission name="l_hip_pitch" />
@@ -67,7 +67,7 @@
     <collision>
       <!-- <xacro:insert_mesh_l_hip_pitch_link /> -->
-      <origin xyz="0.03 -0.05 -0.04" rpy="0.0 0.0 0.0"/>
+      <origin xyz="0 -0.02 -0.04" rpy="0.0 0.0 0.0"/>
       <geometry>
-        <box size="0.03 0.03 0.13"/>
+        <box size="0.033 0.033 0.13"/>
       </geometry>
     </collision>
@@ -83,5 +83,5 @@
     <axis xyz="0 1 0" />
     <limit effort="1.51" velocity="100" lower="${-pi*0.9}" upper="${pi*0.9}" />
-    <dynamics damping="0.01" friction="0.0" />
+    <dynamics damping="0.1" friction="0.0" />
   </joint>
   <xacro:insert_transmission name="l_knee" />
@@ -93,7 +93,7 @@
     <collision>
       <!-- <xacro:insert_mesh_l_knee_link /> -->
-      <origin xyz="0.03 -0.05 -0.05" rpy="0.0 0.0 0.0"/>
+      <origin xyz="0 -0.02 -0.05" rpy="0.0 0.0 0.0"/>
       <geometry>
-        <box size="0.03 0.03 0.1"/>
+        <box size="0.033 0.033 0.1"/>
       </geometry>
     </collision>
@@ -109,5 +109,5 @@
     <axis xyz="0 -1 0" />
     <limit effort="1.51" velocity="100" lower="${-pi*0.9}" upper="${pi*0.9}" />
-    <dynamics damping="0.01" friction="0.0" />
+    <dynamics damping="0.1" friction="0.0" />
   </joint>
   <xacro:insert_transmission name="l_ank_pitch" />
@@ -131,5 +131,5 @@
     <axis xyz="1 0 0" />
     <limit effort="1.51" velocity="100" lower="${-pi*0.9}" upper="${pi*0.9}" />
-    <dynamics damping="0.01" friction="0.0" />
+    <dynamics damping="0.1" friction="0.0" />
   </joint>
   <xacro:insert_transmission name="l_ank_roll" />
@@ -141,7 +141,7 @@
     <collision>
       <!-- <xacro:insert_mesh_l_ank_roll_link /> -->
-      <origin xyz="0 0.03 -0.03" rpy="0 0 0" />
+      <origin xyz="0.02 0.012 -0.03" rpy="0 0 0" />
       <geometry>
-        <box size="0.145 0.09 0.01" />
+        <box size="0.14 0.085 0.01" />
       </geometry>
     </collision>

File: op3_gym/urdf_simple/robotis_op3.structure.rarm.xacro (robot description, xacro)
@@ -13,5 +13,5 @@
     <axis xyz="0 -1 0" />
     <limit effort="1.51" velocity="100" lower="${-pi*0.9}" upper="${pi*0.9}" />
-    <dynamics damping="0.01" friction="0.0" />
+    <dynamics damping="0.1" friction="0.0" />
   </joint>
   <xacro:insert_transmission name="r_sho_pitch" />
@@ -35,5 +35,5 @@
     <axis xyz="-1 0 0" />
     <limit effort="1.51" velocity="100" lower="${-pi*0.9}" upper="${pi*0.9}" />
-    <dynamics damping="0.01" friction="0.0" />
+    <dynamics damping="0.1" friction="0.0" />
   </joint>
   <xacro:insert_transmission name="r_sho_roll" />
@@ -57,5 +57,5 @@
     <axis xyz="1 0 0" />
     <limit effort="1.51" velocity="100" lower="${-pi*0.9}" upper="${pi*0.9}" />
-    <dynamics damping="0.01" friction="0.0" />
+    <dynamics damping="0.1" friction="0.0" />
   </joint>
   <xacro:insert_transmission name="r_el" />

File: op3_gym/urdf_simple/robotis_op3.structure.rleg.xacro (robot description, xacro)
@@ -13,5 +13,5 @@
     <axis xyz="0 0 -1" />
     <limit effort="1.51" velocity="100" lower="${-pi*0.9}" upper="${pi*0.9}" />
-    <dynamics damping="0.01" friction="0.0" />
+    <dynamics damping="0.1" friction="0.0" />
   </joint>
   <xacro:insert_transmission name="r_hip_yaw" />
@@ -35,5 +35,5 @@
     <axis xyz="-1 0 0" />
     <limit effort="1.51" velocity="100" lower="${-pi*0.9}" upper="${pi*0.9}" />
-    <dynamics damping="0.01" friction="0.0" />
+    <dynamics damping="0.1" friction="0.0" />
   </joint>
   <xacro:insert_transmission name="r_hip_roll" />
@@ -57,5 +57,5 @@
     <axis xyz="0 -1 0" />
     <limit effort="1.51" velocity="100" lower="${-pi*0.9}" upper="${pi*0.9}" />
-    <dynamics damping="0.01" friction="0.0" />
+    <dynamics damping="0.1" friction="0.0" />
   </joint>
   <xacro:insert_transmission name="r_hip_pitch" />
@@ -67,7 +67,7 @@
     <collision>
       <!-- <xacro:insert_mesh_r_hip_pitch_link /> -->
-      <origin xyz="0.03 0.0 -0.04" rpy="0.0 0.0 0.0"/>
+      <origin xyz="0 0.022 -0.04" rpy="0.0 0.0 0.0"/>
       <geometry>
-        <box size="0.03 0.03 0.13"/>
+        <box size="0.033 0.033 0.13"/>
       </geometry>
     </collision>
@@ -83,5 +83,5 @@
     <axis xyz="0 -1 0" />
     <limit effort="1.51" velocity="100" lower="${-pi*0.9}" upper="${pi*0.9}" />
-    <dynamics damping="0.01" friction="0.0" />
+    <dynamics damping="0.1" friction="0.0" />
   </joint>
   <xacro:insert_transmission name="r_knee" />
@@ -93,7 +93,7 @@
     <collision>
       <!-- <xacro:insert_mesh_r_knee_link /> -->
-      <origin xyz="0.03 0.0 -0.05" rpy="0.0 0.0 0.0"/>
+      <origin xyz="0 0.022 -0.05" rpy="0.0 0.0 0.0"/>
       <geometry>
-        <box size="0.03 0.03 0.1"/>
+        <box size="0.033 0.033 0.1"/>
       </geometry>
     </collision>
@@ -109,5 +109,5 @@
     <axis xyz="0 1 0" />
     <limit effort="1.51" velocity="100" lower="${-pi*0.9}" upper="${pi*0.9}" />
-    <dynamics damping="0.01" friction="0.0" />
+    <dynamics damping="0.1" friction="0.0" />
   </joint>
   <xacro:insert_transmission name="r_ank_pitch" />
@@ -131,5 +131,5 @@
     <axis xyz="1 0 0" />
     <limit effort="1.51" velocity="100" lower="${-pi*0.9}" upper="${pi*0.9}" />
-    <dynamics damping="0.01" friction="0.0" />
+    <dynamics damping="0.1" friction="0.0" />
   </joint>
   <xacro:insert_transmission name="r_ank_roll" />
@@ -141,7 +141,7 @@
     <collision>
       <!-- <xacro:insert_mesh_r_ank_roll_link /> -->
-      <origin xyz="0 0 -0.03" rpy="0 0 0" />
+      <origin xyz="0.02 -0.01 -0.03" rpy="0 0 0" />
       <geometry>
-        <box size="0.145 0.09 0.01" />
+        <box size="0.14 0.085 0.01" />
       </geometry>
     </collision>

File: op3_gym/urdf_simple/robotis_op3.urdf.xacro (robot description, xacro)
@@ -38,7 +38,7 @@
       <xacro:insert_mesh_body_link />
     </visual>
-    <collision>
+    <!-- <collision>
       <xacro:insert_mesh_body_link />
-    </collision>
+    </collision> -->
     <inertial>
       <xacro:insert_inertia_body_link />
