Commit message: weakened motor strength

File: op3_gym/urdf/robotis_op3.gazebo.xacro (robot description, xacro)
@@ -271,5 +271,5 @@
         <topicName>robotis_op3/imu</topicName>
         <bodyName>body_link</bodyName>
-        <updateRateHZ>10.0</updateRateHZ>
+        <updateRateHZ>60.0</updateRateHZ>
         <gaussianNoise>0.0</gaussianNoise>
         <xyzOffset>0 0 0</xyzOffset>

File: op3_gym/urdf/robotis_op3.structure.head.xacro (robot description, xacro)
@@ -12,5 +12,5 @@
     <origin xyz="-0.001 0.0 0.1365" rpy="0 0 0" />
     <axis xyz="0 0 1" />
-    <limit effort="5" velocity="3" lower="${-pi*0.9}" upper="${pi*0.9}" />
+    <limit effort="5" velocity="1" lower="${-pi*0.9}" upper="${pi*0.9}" />
     <dynamics damping="0.1" friction="0.0" />
   </joint>
@@ -34,5 +34,5 @@
     <origin xyz="0.010 0.019 0.0285" rpy="0 0 0" />
     <axis xyz="0 -1 0" />
-    <limit effort="5" velocity="3" lower="${-pi*0.9}" upper="${pi*0.9}" />
+    <limit effort="5" velocity="1" lower="${-pi*0.9}" upper="${pi*0.9}" />
     <dynamics damping="0.1" friction="0.0" />
   </joint>

File: op3_gym/urdf/robotis_op3.structure.larm.xacro (robot description, xacro)
@@ -12,5 +12,5 @@
     <origin xyz="-0.001 0.06 0.111" rpy="0 0 0" />
     <axis xyz="0 1 0" />
-    <limit effort="5" velocity="3" lower="${-pi*0.9}" upper="${pi*0.9}" />
+    <limit effort="5" velocity="1" lower="${-pi*0.9}" upper="${pi*0.9}" />
     <dynamics damping="0.1" friction="0.0" />
   </joint>
@@ -34,5 +34,5 @@
     <origin xyz="0.019 0.0285 -0.010" rpy="0 0 0" />
     <axis xyz="-1 0 0" />
-    <limit effort="5" velocity="3" lower="${-pi*0.9}" upper="${pi*0.9}" />
+    <limit effort="5" velocity="1" lower="${-pi*0.9}" upper="${pi*0.9}" />
     <dynamics damping="0.1" friction="0.0" />
   </joint>
@@ -56,5 +56,5 @@
     <origin xyz="0.0 0.0904 -0.0001" rpy="0 0 0" />
     <axis xyz="1 0 0" />
-    <limit effort="5" velocity="3" lower="${-pi*0.9}" upper="${pi*0.9}" />
+    <limit effort="5" velocity="1" lower="${-pi*0.9}" upper="${pi*0.9}" />
     <dynamics damping="0.1" friction="0.0" />
   </joint>

File: op3_gym/urdf/robotis_op3.structure.lleg.xacro (robot description, xacro)
@@ -12,5 +12,5 @@
     <origin xyz="0.0 0.035 0.0" rpy="0 0 0" />
     <axis xyz="0 0 -1" />
-    <limit effort="5" velocity="3" lower="${-pi*0.9}" upper="${pi*0.9}" />
+    <limit effort="5" velocity="1" lower="${-pi*0.9}" upper="${pi*0.9}" />
     <dynamics damping="0.1" friction="0.0" />
   </joint>
@@ -34,5 +34,5 @@
     <origin xyz="-0.024 0.0 -0.0285" rpy="0 0 0" />
     <axis xyz="-1 0 0" />
-    <limit effort="5" velocity="3" lower="${-pi*0.9}" upper="${pi*0.9}" />
+    <limit effort="5" velocity="1" lower="${-pi*0.9}" upper="${pi*0.9}" />
     <dynamics damping="0.1" friction="0.0" />
   </joint>
@@ -56,5 +56,5 @@
     <origin xyz="0.0241 0.019 0.0" rpy="0 0 0" />
     <axis xyz="0 1 0" />
-    <limit effort="5" velocity="3" lower="${-pi*0.9}" upper="${pi*0.9}" />
+    <limit effort="5" velocity="1" lower="${-pi*0.9}" upper="${pi*0.9}" />
     <dynamics damping="0.1" friction="0.0" />
   </joint>
@@ -78,5 +78,5 @@
     <origin xyz="0.0 0.0 -0.11015" rpy="0 0 0" />
     <axis xyz="0 1 0" />
-    <limit effort="5" velocity="3" lower="${-pi*0.9}" upper="${pi*0.9}" />
+    <limit effort="5" velocity="1" lower="${-pi*0.9}" upper="${pi*0.9}" />
     <dynamics damping="0.1" friction="0.0" />
   </joint>
@@ -100,5 +100,5 @@
     <origin xyz="0 0 -0.110" rpy="0 0 0" />
     <axis xyz="0 -1 0" />
-    <limit effort="5" velocity="3" lower="${-pi*0.9}" upper="${pi*0.9}" />
+    <limit effort="5" velocity="1" lower="${-pi*0.9}" upper="${pi*0.9}" />
     <dynamics damping="0.1" friction="0.0" />
   </joint>
@@ -122,5 +122,5 @@
     <origin xyz="-0.0241 -0.019 0" rpy="0 0 0" />
     <axis xyz="1 0 0" />
-    <limit effort="5" velocity="3" lower="${-pi*0.9}" upper="${pi*0.9}" />
+    <limit effort="5" velocity="1" lower="${-pi*0.9}" upper="${pi*0.9}" />
     <dynamics damping="0.1" friction="0.0" />
   </joint>

File: op3_gym/urdf/robotis_op3.structure.rarm.xacro (robot description, xacro)
@@ -12,5 +12,5 @@
     <origin xyz="-0.001 -0.06 0.111" rpy="0 0 0" />
     <axis xyz="0 -1 0" />
-    <limit effort="5" velocity="3" lower="${-pi*0.9}" upper="${pi*0.9}" />
+    <limit effort="5" velocity="1" lower="${-pi*0.9}" upper="${pi*0.9}" />
     <dynamics damping="0.1" friction="0.0" />
   </joint>
@@ -34,5 +34,5 @@
     <origin xyz="0.019 -0.0285 -0.010" rpy="0 0 0" />
     <axis xyz="-1 0 0" />
-    <limit effort="5" velocity="3" lower="${-pi*0.9}" upper="${pi*0.9}" />
+    <limit effort="5" velocity="1" lower="${-pi*0.9}" upper="${pi*0.9}" />
     <dynamics damping="0.1" friction="0.0" />
   </joint>
@@ -56,5 +56,5 @@
     <origin xyz="0.0 -0.0904 -0.0001" rpy="0 0 0" />
     <axis xyz="1 0 0" />
-    <limit effort="5" velocity="3" lower="${-pi*0.9}" upper="${pi*0.9}" />
+    <limit effort="5" velocity="1" lower="${-pi*0.9}" upper="${pi*0.9}" />
     <dynamics damping="0.1" friction="0.0" />
   </joint>

File: op3_gym/urdf/robotis_op3.structure.rleg.xacro (robot description, xacro)
@@ -12,5 +12,5 @@
     <origin xyz="0.0 -0.035 0.0" rpy="0 0 0" />
     <axis xyz="0 0 -1" />
-    <limit effort="5" velocity="3" lower="${-pi*0.9}" upper="${pi*0.9}" />
+    <limit effort="5" velocity="1" lower="${-pi*0.9}" upper="${pi*0.9}" />
     <dynamics damping="0.1" friction="0.0" />
   </joint>
@@ -34,5 +34,5 @@
     <origin xyz="-0.024 0.0 -0.0285" rpy="0 0 0" />
     <axis xyz="-1 0 0" />
-    <limit effort="5" velocity="3" lower="${-pi*0.9}" upper="${pi*0.9}" />
+    <limit effort="5" velocity="1" lower="${-pi*0.9}" upper="${pi*0.9}" />
     <dynamics damping="0.1" friction="0.0" />
   </joint>
@@ -56,5 +56,5 @@
     <origin xyz="0.0241 -0.019 0.0" rpy="0 0 0" />
     <axis xyz="0 -1 0" />
-    <limit effort="5" velocity="3" lower="${-pi*0.9}" upper="${pi*0.9}" />
+    <limit effort="5" velocity="1" lower="${-pi*0.9}" upper="${pi*0.9}" />
     <dynamics damping="0.1" friction="0.0" />
   </joint>
@@ -78,5 +78,5 @@
     <origin xyz="0.0 0.0 -0.11015" rpy="0 0 0" />
     <axis xyz="0 -1 0" />
-    <limit effort="5" velocity="3" lower="${-pi*0.9}" upper="${pi*0.9}" />
+    <limit effort="5" velocity="1" lower="${-pi*0.9}" upper="${pi*0.9}" />
     <dynamics damping="0.1" friction="0.0" />
   </joint>
@@ -100,5 +100,5 @@
     <origin xyz="0 0 -0.110" rpy="0 0 0" />
     <axis xyz="0 1 0" />
-    <limit effort="5" velocity="3" lower="${-pi*0.9}" upper="${pi*0.9}" />
+    <limit effort="5" velocity="1" lower="${-pi*0.9}" upper="${pi*0.9}" />
     <dynamics damping="0.1" friction="0.0" />
   </joint>
@@ -122,5 +122,5 @@
     <origin xyz="-0.0241 0.019 0" rpy="0 0 0" />
     <axis xyz="1 0 0" />
-    <limit effort="5" velocity="3" lower="${-pi*0.9}" upper="${pi*0.9}" />
+    <limit effort="5" velocity="1" lower="${-pi*0.9}" upper="${pi*0.9}" />
     <dynamics damping="0.1" friction="0.0" />
   </joint>

File: op3_gym/urdf/robotis_op3.urdf.xacro (robot description, xacro)
@@ -1,15 +1,15 @@
 <?xml version="1.0" ?>
 <robot xmlns:xacro="http://ros.org/wiki/xacro" name="robotis_op3">
-  <xacro:include filename="$(find op3_description)/urdf/robotis_op3.visuals.xacro" />
-  <xacro:include filename="$(find op3_description)/urdf/robotis_op3.inertia.xacro" />
-  <xacro:include filename="$(find op3_description)/urdf/robotis_op3.structure.rleg.xacro" />
-  <xacro:include filename="$(find op3_description)/urdf/robotis_op3.structure.lleg.xacro" />
-  <xacro:include filename="$(find op3_description)/urdf/robotis_op3.structure.rarm.xacro" />
-  <xacro:include filename="$(find op3_description)/urdf/robotis_op3.structure.larm.xacro" />
-  <xacro:include filename="$(find op3_description)/urdf/robotis_op3.structure.head.xacro" />
-  <xacro:include filename="$(find op3_description)/urdf/robotis_op3.gazebo.xacro" />
-  <xacro:include filename="$(find op3_description)/urdf/robotis_op3.transmissions.xacro" />
+  <xacro:include filename="$(find op3_gym)/urdf/robotis_op3.visuals.xacro" />
+  <xacro:include filename="$(find op3_gym)/urdf/robotis_op3.inertia.xacro" />
+  <xacro:include filename="$(find op3_gym)/urdf/robotis_op3.structure.rleg.xacro" />
+  <xacro:include filename="$(find op3_gym)/urdf/robotis_op3.structure.lleg.xacro" />
+  <xacro:include filename="$(find op3_gym)/urdf/robotis_op3.structure.rarm.xacro" />
+  <xacro:include filename="$(find op3_gym)/urdf/robotis_op3.structure.larm.xacro" />
+  <xacro:include filename="$(find op3_gym)/urdf/robotis_op3.structure.head.xacro" />
+  <xacro:include filename="$(find op3_gym)/urdf/robotis_op3.gazebo.xacro" />
+  <xacro:include filename="$(find op3_gym)/urdf/robotis_op3.transmissions.xacro" />
   <!--
-  <xacro:include filename="$(find op3_description)/urdf/gazebo_harness.xacro" />
+  <xacro:include filename="$(find op3_gym)/urdf/gazebo_harness.xacro" />
   -->
   <!-- harness link -->

Commit message: Fixed IMU lastest time problem

File: op3_gym/urdf/robotis_op3.gazebo.xacro (robot description, xacro)
@@ -11,5 +11,5 @@
     <mu2>0.2</mu2>
     <material>Gazebo/White</material>
-    <selfCollide>false</selfCollide>
+    <selfCollide>true</selfCollide>
   </gazebo>
   <!-- left leg links -->
@@ -18,5 +18,5 @@
     <mu2>0.2</mu2>
     <material>Gazebo/White</material>
-    <selfCollide>false</selfCollide>
+    <selfCollide>true</selfCollide>
   </gazebo>
   <gazebo reference="l_hip_roll_link">
@@ -24,5 +24,5 @@
     <mu2>0.2</mu2>
     <material>Gazebo/White</material>
-    <selfCollide>false</selfCollide>
+    <selfCollide>true</selfCollide>
   </gazebo>
   <gazebo reference="l_hip_pitch_link">
@@ -30,5 +30,5 @@
     <mu2>0.2</mu2>
     <material>Gazebo/White</material>
-    <selfCollide>false</selfCollide>
+    <selfCollide>true</selfCollide>
   </gazebo>
   <gazebo reference="l_knee_link">
@@ -36,5 +36,5 @@
     <mu2>0.2</mu2>
     <material>Gazebo/White</material>
-    <selfCollide>false</selfCollide>
+    <selfCollide>true</selfCollide>
   </gazebo>
   <gazebo reference="l_ank_pitch_link">
@@ -42,5 +42,5 @@
     <mu2>0.2</mu2>
     <material>Gazebo/White</material>
-    <selfCollide>false</selfCollide>
+    <selfCollide>true</selfCollide>
   </gazebo>
   <gazebo reference="l_ank_roll_link">
@@ -59,5 +59,5 @@
     <mu2>0.2</mu2>
     <material>Gazebo/White</material>
-    <selfCollide>false</selfCollide>
+    <selfCollide>true</selfCollide>
   </gazebo>
   <gazebo reference="r_hip_roll_link">
@@ -65,5 +65,5 @@
     <mu2>0.2</mu2>
     <material>Gazebo/White</material>
-    <selfCollide>false</selfCollide>
+    <selfCollide>true</selfCollide>
   </gazebo>
   <gazebo reference="r_hip_pitch_link">
@@ -71,5 +71,5 @@
     <mu2>0.2</mu2>
     <material>Gazebo/White</material>
-    <selfCollide>false</selfCollide>
+    <selfCollide>true</selfCollide>
   </gazebo>
   <gazebo reference="r_knee_link">
@@ -77,5 +77,5 @@
     <mu2>0.2</mu2>
     <material>Gazebo/White</material>
-    <selfCollide>false</selfCollide>
+    <selfCollide>true</selfCollide>
   </gazebo>
   <gazebo reference="r_ank_pitch_link">
@@ -83,5 +83,5 @@
     <mu2>0.2</mu2>
     <material>Gazebo/White</material>
-    <selfCollide>false</selfCollide>
+    <selfCollide>true</selfCollide>
   </gazebo>
   <gazebo reference="r_ank_roll_link">
@@ -100,5 +100,5 @@
     <mu2>0.2</mu2>
     <material>Gazebo/White</material>
-    <selfCollide>false</selfCollide>
+    <selfCollide>true</selfCollide>
   </gazebo>
   <gazebo reference="r_sho_roll_link">
@@ -106,5 +106,5 @@
     <mu2>0.2</mu2>
     <material>Gazebo/White</material>
-    <selfCollide>false</selfCollide>
+    <selfCollide>true</selfCollide>
   </gazebo>
   <gazebo reference="r_el_link">
@@ -112,5 +112,5 @@
     <mu2>0.2</mu2>
     <material>Gazebo/White</material>
-    <selfCollide>false</selfCollide>
+    <selfCollide>true</selfCollide>
   </gazebo>
   <gazebo reference="l_sho_pitch_link">
@@ -118,5 +118,5 @@
     <mu2>0.2</mu2>
     <material>Gazebo/White</material>
-    <selfCollide>false</selfCollide>
+    <selfCollide>true</selfCollide>
   </gazebo>
   <gazebo reference="l_sho_roll_link">
@@ -124,5 +124,5 @@
     <mu2>0.2</mu2>
     <material>Gazebo/White</material>
-    <selfCollide>false</selfCollide>
+    <selfCollide>true</selfCollide>
   </gazebo>
   <gazebo reference="l_el_link">
@@ -130,5 +130,5 @@
     <mu2>0.2</mu2>
     <material>Gazebo/White</material>
-    <selfCollide>false</selfCollide>
+    <selfCollide>true</selfCollide>
   </gazebo>
   <gazebo reference="head_pan_link">
@@ -136,5 +136,5 @@
     <mu2>0.2</mu2>
     <material>Gazebo/White</material>
-    <selfCollide>false</selfCollide>
+    <selfCollide>true</selfCollide>
   </gazebo>
   <gazebo reference="head_tilt_link">
@@ -142,5 +142,5 @@
     <mu2>0.2</mu2>
     <material>Gazebo/White</material>
-    <selfCollide>false</selfCollide>
+    <selfCollide>true</selfCollide>
   </gazebo>
 <!--
@@ -271,5 +271,5 @@
         <topicName>robotis_op3/imu</topicName>
         <bodyName>body_link</bodyName>
-        <updateRateHZ>60.0</updateRateHZ>
+        <updateRateHZ>0</updateRateHZ>
         <gaussianNoise>0.0</gaussianNoise>
         <xyzOffset>0 0 0</xyzOffset>

File: op3_gym/urdf/robotis_op3.structure.head.xacro (robot description, xacro)
@@ -12,5 +12,5 @@
     <origin xyz="-0.001 0.0 0.1365" rpy="0 0 0" />
     <axis xyz="0 0 1" />
-    <limit effort="5" velocity="1" lower="${-pi*0.9}" upper="${pi*0.9}" />
+    <limit effort="5" velocity="5" lower="${-pi*0.9}" upper="${pi*0.9}" />
     <dynamics damping="0.1" friction="0.0" />
   </joint>
@@ -34,5 +34,5 @@
     <origin xyz="0.010 0.019 0.0285" rpy="0 0 0" />
     <axis xyz="0 -1 0" />
-    <limit effort="5" velocity="1" lower="${-pi*0.9}" upper="${pi*0.9}" />
+    <limit effort="5" velocity="5" lower="${-pi*0.9}" upper="${pi*0.9}" />
     <dynamics damping="0.1" friction="0.0" />
   </joint>

File: op3_gym/urdf/robotis_op3.structure.larm.xacro (robot description, xacro)
@@ -12,6 +12,6 @@
     <origin xyz="-0.001 0.06 0.111" rpy="0 0 0" />
     <axis xyz="0 1 0" />
-    <limit effort="5" velocity="1" lower="${-pi*0.9}" upper="${pi*0.9}" />
-    <dynamics damping="0.1" friction="0.0" />
+    <limit effort="5" velocity="5" lower="${-pi*0.9}" upper="${pi*0.9}" />
+    <dynamics damping="0.1" friction="0.01" />
   </joint>
   <xacro:insert_transmission name="l_sho_pitch" />
@@ -34,6 +34,6 @@
     <origin xyz="0.019 0.0285 -0.010" rpy="0 0 0" />
     <axis xyz="-1 0 0" />
-    <limit effort="5" velocity="1" lower="${-pi*0.9}" upper="${pi*0.9}" />
-    <dynamics damping="0.1" friction="0.0" />
+    <limit effort="5" velocity="5" lower="${-pi*0.9}" upper="${pi*0.9}" />
+    <dynamics damping="0.1" friction="0.01" />
   </joint>
   <xacro:insert_transmission name="l_sho_roll" />
@@ -56,6 +56,6 @@
     <origin xyz="0.0 0.0904 -0.0001" rpy="0 0 0" />
     <axis xyz="1 0 0" />
-    <limit effort="5" velocity="1" lower="${-pi*0.9}" upper="${pi*0.9}" />
-    <dynamics damping="0.1" friction="0.0" />
+    <limit effort="5" velocity="5" lower="${-pi*0.9}" upper="${pi*0.9}" />
+    <dynamics damping="0.1" friction="0.01" />
   </joint>
   <xacro:insert_transmission name="l_el" />

File: op3_gym/urdf/robotis_op3.structure.lleg.xacro (robot description, xacro)
@@ -12,5 +12,5 @@
     <origin xyz="0.0 0.035 0.0" rpy="0 0 0" />
     <axis xyz="0 0 -1" />
-    <limit effort="5" velocity="1" lower="${-pi*0.9}" upper="${pi*0.9}" />
+    <limit effort="5" velocity="5" lower="${-pi*0.9}" upper="${pi*0.9}" />
     <dynamics damping="0.1" friction="0.0" />
   </joint>
@@ -34,5 +34,5 @@
     <origin xyz="-0.024 0.0 -0.0285" rpy="0 0 0" />
     <axis xyz="-1 0 0" />
-    <limit effort="5" velocity="1" lower="${-pi*0.9}" upper="${pi*0.9}" />
+    <limit effort="5" velocity="5" lower="${-pi*0.9}" upper="${pi*0.9}" />
     <dynamics damping="0.1" friction="0.0" />
   </joint>
@@ -56,5 +56,5 @@
     <origin xyz="0.0241 0.019 0.0" rpy="0 0 0" />
     <axis xyz="0 1 0" />
-    <limit effort="5" velocity="1" lower="${-pi*0.9}" upper="${pi*0.9}" />
+    <limit effort="5" velocity="5" lower="${-pi*0.9}" upper="${pi*0.9}" />
     <dynamics damping="0.1" friction="0.0" />
   </joint>
@@ -78,5 +78,5 @@
     <origin xyz="0.0 0.0 -0.11015" rpy="0 0 0" />
     <axis xyz="0 1 0" />
-    <limit effort="5" velocity="1" lower="${-pi*0.9}" upper="${pi*0.9}" />
+    <limit effort="5" velocity="5" lower="${-pi*0.9}" upper="${pi*0.9}" />
     <dynamics damping="0.1" friction="0.0" />
   </joint>
@@ -100,5 +100,5 @@
     <origin xyz="0 0 -0.110" rpy="0 0 0" />
     <axis xyz="0 -1 0" />
-    <limit effort="5" velocity="1" lower="${-pi*0.9}" upper="${pi*0.9}" />
+    <limit effort="5" velocity="5" lower="${-pi*0.9}" upper="${pi*0.9}" />
     <dynamics damping="0.1" friction="0.0" />
   </joint>
@@ -122,5 +122,5 @@
     <origin xyz="-0.0241 -0.019 0" rpy="0 0 0" />
     <axis xyz="1 0 0" />
-    <limit effort="5" velocity="1" lower="${-pi*0.9}" upper="${pi*0.9}" />
+    <limit effort="5" velocity="5" lower="${-pi*0.9}" upper="${pi*0.9}" />
     <dynamics damping="0.1" friction="0.0" />
   </joint>

File: op3_gym/urdf/robotis_op3.structure.rarm.xacro (robot description, xacro)
@@ -12,5 +12,5 @@
     <origin xyz="-0.001 -0.06 0.111" rpy="0 0 0" />
     <axis xyz="0 -1 0" />
-    <limit effort="5" velocity="1" lower="${-pi*0.9}" upper="${pi*0.9}" />
+    <limit effort="5" velocity="5" lower="${-pi*0.9}" upper="${pi*0.9}" />
     <dynamics damping="0.1" friction="0.0" />
   </joint>
@@ -34,5 +34,5 @@
     <origin xyz="0.019 -0.0285 -0.010" rpy="0 0 0" />
     <axis xyz="-1 0 0" />
-    <limit effort="5" velocity="1" lower="${-pi*0.9}" upper="${pi*0.9}" />
+    <limit effort="5" velocity="5" lower="${-pi*0.9}" upper="${pi*0.9}" />
     <dynamics damping="0.1" friction="0.0" />
   </joint>
@@ -56,5 +56,5 @@
     <origin xyz="0.0 -0.0904 -0.0001" rpy="0 0 0" />
     <axis xyz="1 0 0" />
-    <limit effort="5" velocity="1" lower="${-pi*0.9}" upper="${pi*0.9}" />
+    <limit effort="5" velocity="5" lower="${-pi*0.9}" upper="${pi*0.9}" />
     <dynamics damping="0.1" friction="0.0" />
   </joint>

File: op3_gym/urdf/robotis_op3.structure.rleg.xacro (robot description, xacro)
@@ -12,5 +12,5 @@
     <origin xyz="0.0 -0.035 0.0" rpy="0 0 0" />
     <axis xyz="0 0 -1" />
-    <limit effort="5" velocity="1" lower="${-pi*0.9}" upper="${pi*0.9}" />
+    <limit effort="5" velocity="5" lower="${-pi*0.9}" upper="${pi*0.9}" />
     <dynamics damping="0.1" friction="0.0" />
   </joint>
@@ -34,5 +34,5 @@
     <origin xyz="-0.024 0.0 -0.0285" rpy="0 0 0" />
     <axis xyz="-1 0 0" />
-    <limit effort="5" velocity="1" lower="${-pi*0.9}" upper="${pi*0.9}" />
+    <limit effort="5" velocity="5" lower="${-pi*0.9}" upper="${pi*0.9}" />
     <dynamics damping="0.1" friction="0.0" />
   </joint>
@@ -56,5 +56,5 @@
     <origin xyz="0.0241 -0.019 0.0" rpy="0 0 0" />
     <axis xyz="0 -1 0" />
-    <limit effort="5" velocity="1" lower="${-pi*0.9}" upper="${pi*0.9}" />
+    <limit effort="5" velocity="5" lower="${-pi*0.9}" upper="${pi*0.9}" />
     <dynamics damping="0.1" friction="0.0" />
   </joint>
@@ -78,5 +78,5 @@
     <origin xyz="0.0 0.0 -0.11015" rpy="0 0 0" />
     <axis xyz="0 -1 0" />
-    <limit effort="5" velocity="1" lower="${-pi*0.9}" upper="${pi*0.9}" />
+    <limit effort="5" velocity="5" lower="${-pi*0.9}" upper="${pi*0.9}" />
     <dynamics damping="0.1" friction="0.0" />
   </joint>
@@ -100,5 +100,5 @@
     <origin xyz="0 0 -0.110" rpy="0 0 0" />
     <axis xyz="0 1 0" />
-    <limit effort="5" velocity="1" lower="${-pi*0.9}" upper="${pi*0.9}" />
+    <limit effort="5" velocity="5" lower="${-pi*0.9}" upper="${pi*0.9}" />
     <dynamics damping="0.1" friction="0.0" />
   </joint>
@@ -122,5 +122,5 @@
     <origin xyz="-0.0241 0.019 0" rpy="0 0 0" />
     <axis xyz="1 0 0" />
-    <limit effort="5" velocity="1" lower="${-pi*0.9}" upper="${pi*0.9}" />
+    <limit effort="5" velocity="5" lower="${-pi*0.9}" upper="${pi*0.9}" />
     <dynamics damping="0.1" friction="0.0" />
   </joint>
