Commit message: checkpoint 210527

File: op3_gym/urdf/robotis_op3.gazebo.xacro (robot description, xacro)
@@ -11,5 +11,5 @@
     <mu2>0.2</mu2>
     <material>Gazebo/White</material>
-    <selfCollide>true</selfCollide>
+    <selfCollide>false</selfCollide>
   </gazebo>
   <!-- left leg links -->
@@ -18,5 +18,5 @@
     <mu2>0.2</mu2>
     <material>Gazebo/White</material>
-    <selfCollide>true</selfCollide>
+    <selfCollide>false</selfCollide>
   </gazebo>
   <gazebo reference="l_hip_roll_link">
@@ -24,5 +24,5 @@
     <mu2>0.2</mu2>
     <material>Gazebo/White</material>
-    <selfCollide>true</selfCollide>
+    <selfCollide>false</selfCollide>
   </gazebo>
   <gazebo reference="l_hip_pitch_link">
@@ -30,5 +30,5 @@
     <mu2>0.2</mu2>
     <material>Gazebo/White</material>
-    <selfCollide>true</selfCollide>
+    <selfCollide>false</selfCollide>
   </gazebo>
   <gazebo reference="l_knee_link">
@@ -36,5 +36,5 @@
     <mu2>0.2</mu2>
     <material>Gazebo/White</material>
-    <selfCollide>true</selfCollide>
+    <selfCollide>false</selfCollide>
   </gazebo>
   <gazebo reference="l_ank_pitch_link">
@@ -42,5 +42,5 @@
     <mu2>0.2</mu2>
     <material>Gazebo/White</material>
-    <selfCollide>true</selfCollide>
+    <selfCollide>false</selfCollide>
   </gazebo>
   <gazebo reference="l_ank_roll_link">
@@ -59,5 +59,5 @@
     <mu2>0.2</mu2>
     <material>Gazebo/White</material>
-    <selfCollide>true</selfCollide>
+    <selfCollide>false</selfCollide>
   </gazebo>
   <gazebo reference="r_hip_roll_link">
@@ -65,5 +65,5 @@
     <mu2>0.2</mu2>
     <material>Gazebo/White</material>
-    <selfCollide>true</selfCollide>
+    <selfCollide>false</selfCollide>
   </gazebo>
   <gazebo reference="r_hip_pitch_link">
@@ -71,5 +71,5 @@
     <mu2>0.2</mu2>
     <material>Gazebo/White</material>
-    <selfCollide>true</selfCollide>
+    <selfCollide>false</selfCollide>
   </gazebo>
   <gazebo reference="r_knee_link">
@@ -77,5 +77,5 @@
     <mu2>0.2</mu2>
     <material>Gazebo/White</material>
-    <selfCollide>true</selfCollide>
+    <selfCollide>false</selfCollide>
   </gazebo>
   <gazebo reference="r_ank_pitch_link">
@@ -83,5 +83,5 @@
     <mu2>0.2</mu2>
     <material>Gazebo/White</material>
-    <selfCollide>true</selfCollide>
+    <selfCollide>false</selfCollide>
   </gazebo>
   <gazebo reference="r_ank_roll_link">
@@ -100,5 +100,5 @@
     <mu2>0.2</mu2>
     <material>Gazebo/White</material>
-    <selfCollide>true</selfCollide>
+    <selfCollide>false</selfCollide>
   </gazebo>
   <gazebo reference="r_sho_roll_link">
@@ -106,5 +106,5 @@
     <mu2>0.2</mu2>
     <material>Gazebo/White</material>
-    <selfCollide>true</selfCollide>
+    <selfCollide>false</selfCollide>
   </gazebo>
   <gazebo reference="r_el_link">
@@ -112,5 +112,5 @@
     <mu2>0.2</mu2>
     <material>Gazebo/White</material>
-    <selfCollide>true</selfCollide>
+    <selfCollide>false</selfCollide>
   </gazebo>
   <gazebo reference="l_sho_pitch_link">
@@ -118,5 +118,5 @@
     <mu2>0.2</mu2>
     <material>Gazebo/White</material>
-    <selfCollide>true</selfCollide>
+    <selfCollide>false</selfCollide>
   </gazebo>
   <gazebo reference="l_sho_roll_link">
@@ -124,5 +124,5 @@
     <mu2>0.2</mu2>
     <material>Gazebo/White</material>
-    <selfCollide>true</selfCollide>
+    <selfCollide>false</selfCollide>
   </gazebo>
   <gazebo reference="l_el_link">
@@ -130,5 +130,5 @@
     <mu2>0.2</mu2>
     <material>Gazebo/White</material>
-    <selfCollide>true</selfCollide>
+    <selfCollide>false</selfCollide>
   </gazebo>
   <gazebo reference="head_pan_link">
@@ -136,5 +136,5 @@
     <mu2>0.2</mu2>
     <material>Gazebo/White</material>
-    <selfCollide>true</selfCollide>
+    <selfCollide>false</selfCollide>
   </gazebo>
   <gazebo reference="head_tilt_link">
@@ -142,5 +142,5 @@
     <mu2>0.2</mu2>
     <material>Gazebo/White</material>
-    <selfCollide>true</selfCollide>
+    <selfCollide>false</selfCollide>
   </gazebo>
 <!--
@@ -227,5 +227,5 @@
 -->
   <!-- head camera -->
-  <gazebo reference="cam_gazebo_link">
+  <!-- <gazebo reference="cam_gazebo_link">
     <sensor name='camera' type='camera'>
       <pose>-0.050000 -0.010000 0.000000 -1.5708 0.000000 -3.141592</pose>
@@ -259,5 +259,5 @@
       </plugin>
     </sensor>
-  </gazebo>
+  </gazebo> -->
   <!-- imu sensor -->
   <gazebo reference="body_link">

File: op3_gym/urdf/robotis_op3.structure.head.xacro (robot description, xacro)
@@ -12,5 +12,5 @@
     <origin xyz="-0.001 0.0 0.1365" rpy="0 0 0" />
     <axis xyz="0 0 1" />
-    <limit effort="10" velocity="10" lower="${-pi*0.9}" upper="${pi*0.9}" />
+    <limit effort="5" velocity="0.1" lower="${-pi*0.9}" upper="${pi*0.9}" />
     <dynamics damping="0.1" friction="0.0" />
   </joint>
@@ -34,5 +34,5 @@
     <origin xyz="0.010 0.019 0.0285" rpy="0 0 0" />
     <axis xyz="0 -1 0" />
-    <limit effort="10" velocity="10" lower="${-pi*0.9}" upper="${pi*0.9}" />
+    <limit effort="5" velocity="0.1" lower="${-pi*0.9}" upper="${pi*0.9}" />
     <dynamics damping="0.1" friction="0.0" />
   </joint>
@@ -51,20 +51,20 @@
   </link>
   <!-- camera joint -->
-  <joint name="cam" type="fixed">
-    <origin xyz="0.01425 -0.019 0.04975" rpy="${-pi*0.5} 0 ${-pi*0.5}"/>
-    <parent link="head_tilt_link"/>
-    <child link="cam_link"/>
-  </joint>
-  <joint name="cam_gazebo" type="fixed">
-    <origin xyz="0.01425 -0.019 0.04975" rpy="0 0 0"/>
-    <parent link="head_tilt_link"/>
-    <child link="cam_gazebo_link"/>
-  </joint>
-  <!-- camera link -->
-  <link name="cam_link">
-  </link>
-  <!-- camera link -->
-  <link name="cam_gazebo_link">
-  </link>
+  <!--
+    <joint name="cam" type="fixed">
+      <origin xyz="0.01425 -0.019 0.04975" rpy="${-pi*0.5} 0 ${-pi*0.5}"/>
+      <parent link="head_tilt_link"/>
+      <child link="cam_link"/>
+    </joint>
+    <joint name="cam_gazebo" type="fixed">
+      <origin xyz="0.01425 -0.019 0.04975" rpy="0 0 0"/>
+      <parent link="head_tilt_link"/>
+      <child link="cam_gazebo_link"/>
+    </joint>
+    <link name="cam_link">
+    </link>
+    <link name="cam_gazebo_link">
+    </link>
+  -->
   </xacro:macro>
 </robot>

File: op3_gym/urdf/robotis_op3.structure.larm.xacro (robot description, xacro)
@@ -12,5 +12,5 @@
     <origin xyz="-0.001 0.06 0.111" rpy="0 0 0" />
     <axis xyz="0 1 0" />
-    <limit effort="10" velocity="10" lower="${-pi*0.9}" upper="${pi*0.9}" />
+    <limit effort="5" velocity="0.1" lower="${-pi*0.9}" upper="${pi*0.9}" />
     <dynamics damping="0.1" friction="0.01" />
   </joint>
@@ -34,5 +34,5 @@
     <origin xyz="0.019 0.0285 -0.010" rpy="0 0 0" />
     <axis xyz="-1 0 0" />
-    <limit effort="10" velocity="10" lower="${-pi*0.9}" upper="${pi*0.9}" />
+    <limit effort="5" velocity="0.1" lower="${-pi*0.9}" upper="${pi*0.9}" />
     <dynamics damping="0.1" friction="0.01" />
   </joint>
@@ -56,5 +56,5 @@
     <origin xyz="0.0 0.0904 -0.0001" rpy="0 0 0" />
     <axis xyz="1 0 0" />
-    <limit effort="10" velocity="10" lower="${-pi*0.9}" upper="${pi*0.9}" />
+    <limit effort="5" velocity="0.1" lower="${-pi*0.9}" upper="${pi*0.9}" />
     <dynamics damping="0.1" friction="0.01" />
   </joint>

File: op3_gym/urdf/robotis_op3.structure.lleg.xacro (robot description, xacro)
@@ -12,5 +12,5 @@
     <origin xyz="0.0 0.035 0.0" rpy="0 0 0" />
     <axis xyz="0 0 -1" />
-    <limit effort="10" velocity="10" lower="${-pi*0.9}" upper="${pi*0.9}" />
+    <limit effort="7" velocity="0.1" lower="${-pi*0.9}" upper="${pi*0.9}" />
     <dynamics damping="0.1" friction="0.0" />
   </joint>
@@ -34,5 +34,5 @@
     <origin xyz="-0.024 0.0 -0.0285" rpy="0 0 0" />
     <axis xyz="-1 0 0" />
-    <limit effort="10" velocity="10" lower="${-pi*0.9}" upper="${pi*0.9}" />
+    <limit effort="7" velocity="0.1" lower="${-pi*0.9}" upper="${pi*0.9}" />
     <dynamics damping="0.1" friction="0.0" />
   </joint>
@@ -56,5 +56,5 @@
     <origin xyz="0.0241 0.019 0.0" rpy="0 0 0" />
     <axis xyz="0 1 0" />
-    <limit effort="10" velocity="10" lower="${-pi*0.9}" upper="${pi*0.9}" />
+    <limit effort="7" velocity="0.1" lower="${-pi*0.9}" upper="${pi*0.9}" />
     <dynamics damping="0.1" friction="0.0" />
   </joint>
@@ -78,5 +78,5 @@
     <origin xyz="0.0 0.0 -0.11015" rpy="0 0 0" />
     <axis xyz="0 1 0" />
-    <limit effort="10" velocity="10" lower="${-pi*0.9}" upper="${pi*0.9}" />
+    <limit effort="7" velocity="0.1" lower="${-pi*0.9}" upper="${pi*0.9}" />
     <dynamics damping="0.1" friction="0.0" />
   </joint>
@@ -100,5 +100,5 @@
     <origin xyz="0 0 -0.110" rpy="0 0 0" />
     <axis xyz="0 -1 0" />
-    <limit effort="10" velocity="10" lower="${-pi*0.9}" upper="${pi*0.9}" />
+    <limit effort="7" velocity="0.1" lower="${-pi*0.9}" upper="${pi*0.9}" />
     <dynamics damping="0.1" friction="0.0" />
   </joint>
@@ -122,5 +122,5 @@
     <origin xyz="-0.0241 -0.019 0" rpy="0 0 0" />
     <axis xyz="1 0 0" />
-    <limit effort="10" velocity="10" lower="${-pi*0.9}" upper="${pi*0.9}" />
+    <limit effort="7" velocity="0.1" lower="${-pi*0.9}" upper="${pi*0.9}" />
     <dynamics damping="0.1" friction="0.0" />
   </joint>

File: op3_gym/urdf/robotis_op3.structure.rarm.xacro (robot description, xacro)
@@ -12,5 +12,5 @@
     <origin xyz="-0.001 -0.06 0.111" rpy="0 0 0" />
     <axis xyz="0 -1 0" />
-    <limit effort="10" velocity="10" lower="${-pi*0.9}" upper="${pi*0.9}" />
+    <limit effort="5" velocity="0.1" lower="${-pi*0.9}" upper="${pi*0.9}" />
     <dynamics damping="0.1" friction="0.0" />
   </joint>
@@ -34,5 +34,5 @@
     <origin xyz="0.019 -0.0285 -0.010" rpy="0 0 0" />
     <axis xyz="-1 0 0" />
-    <limit effort="10" velocity="10" lower="${-pi*0.9}" upper="${pi*0.9}" />
+    <limit effort="5" velocity="0.1" lower="${-pi*0.9}" upper="${pi*0.9}" />
     <dynamics damping="0.1" friction="0.0" />
   </joint>
@@ -56,5 +56,5 @@
     <origin xyz="0.0 -0.0904 -0.0001" rpy="0 0 0" />
     <axis xyz="1 0 0" />
-    <limit effort="10" velocity="10" lower="${-pi*0.9}" upper="${pi*0.9}" />
+    <limit effort="5" velocity="0.1" lower="${-pi*0.9}" upper="${pi*0.9}" />
     <dynamics damping="0.1" friction="0.0" />
   </joint>

File: op3_gym/urdf/robotis_op3.structure.rleg.xacro (robot description, xacro)
@@ -12,5 +12,5 @@
     <origin xyz="0.0 -0.035 0.0" rpy="0 0 0" />
     <axis xyz="0 0 -1" />
-    <limit effort="10" velocity="10" lower="${-pi*0.9}" upper="${pi*0.9}" />
+    <limit effort="7" velocity="0.1" lower="${-pi*0.9}" upper="${pi*0.9}" />
     <dynamics damping="0.1" friction="0.0" />
   </joint>
@@ -34,5 +34,5 @@
     <origin xyz="-0.024 0.0 -0.0285" rpy="0 0 0" />
     <axis xyz="-1 0 0" />
-    <limit effort="10" velocity="10" lower="${-pi*0.9}" upper="${pi*0.9}" />
+    <limit effort="7" velocity="0.1" lower="${-pi*0.9}" upper="${pi*0.9}" />
     <dynamics damping="0.1" friction="0.0" />
   </joint>
@@ -56,5 +56,5 @@
     <origin xyz="0.0241 -0.019 0.0" rpy="0 0 0" />
     <axis xyz="0 -1 0" />
-    <limit effort="10" velocity="10" lower="${-pi*0.9}" upper="${pi*0.9}" />
+    <limit effort="7" velocity="0.1" lower="${-pi*0.9}" upper="${pi*0.9}" />
     <dynamics damping="0.1" friction="0.0" />
   </joint>
@@ -78,5 +78,5 @@
     <origin xyz="0.0 0.0 -0.11015" rpy="0 0 0" />
     <axis xyz="0 -1 0" />
-    <limit effort="10" velocity="10" lower="${-pi*0.9}" upper="${pi*0.9}" />
+    <limit effort="7" velocity="0.1" lower="${-pi*0.9}" upper="${pi*0.9}" />
     <dynamics damping="0.1" friction="0.0" />
   </joint>
@@ -100,5 +100,5 @@
     <origin xyz="0 0 -0.110" rpy="0 0 0" />
     <axis xyz="0 1 0" />
-    <limit effort="10" velocity="10" lower="${-pi*0.9}" upper="${pi*0.9}" />
+    <limit effort="7" velocity="0.1" lower="${-pi*0.9}" upper="${pi*0.9}" />
     <dynamics damping="0.1" friction="0.0" />
   </joint>
@@ -122,5 +122,5 @@
     <origin xyz="-0.0241 0.019 0" rpy="0 0 0" />
     <axis xyz="1 0 0" />
-    <limit effort="10" velocity="10" lower="${-pi*0.9}" upper="${pi*0.9}" />
+    <limit effort="7" velocity="0.1" lower="${-pi*0.9}" upper="${pi*0.9}" />
     <dynamics damping="0.1" friction="0.0" />
   </joint>
