Commit message: config checkpoint 210805

File: op3_gym/urdf/robotis_op3.gazebo.xacro (robot description, xacro)
@@ -265,5 +265,5 @@
     <sensor name="imu_sensor" type="imu">
       <always_on>true</always_on>
-      <update_rate>400</update_rate>
+      <update_rate>200</update_rate>
       <visualize>true</visualize>
       <topic>__default_topic__</topic>

File: op3_gym/urdf_simple/robotis_op3.gazebo.xacro (robot description, xacro)
@@ -11,5 +11,5 @@
     <mu2>0.2</mu2>
     <material>Gazebo/White</material>
-    <selfCollide>false</selfCollide>
+    <selfCollide>true</selfCollide>
   </gazebo>
   <!-- left leg links -->
@@ -18,5 +18,5 @@
     <mu2>0.2</mu2>
     <material>Gazebo/White</material>
-    <selfCollide>false</selfCollide>
+    <selfCollide>true</selfCollide>
   </gazebo>
   <gazebo reference="l_hip_roll_link">
@@ -24,5 +24,5 @@
     <mu2>0.2</mu2>
     <material>Gazebo/White</material>
-    <selfCollide>false</selfCollide>
+    <selfCollide>true</selfCollide>
   </gazebo>
   <gazebo reference="l_hip_pitch_link">
@@ -30,5 +30,5 @@
     <mu2>0.2</mu2>
     <material>Gazebo/White</material>
-    <selfCollide>false</selfCollide>
+    <selfCollide>true</selfCollide>
   </gazebo>
   <gazebo reference="l_knee_link">
@@ -36,5 +36,5 @@
     <mu2>0.2</mu2>
     <material>Gazebo/White</material>
-    <selfCollide>false</selfCollide>
+    <selfCollide>true</selfCollide>
   </gazebo>
   <gazebo reference="l_ank_pitch_link">
@@ -42,5 +42,5 @@
     <mu2>0.2</mu2>
     <material>Gazebo/White</material>
-    <selfCollide>false</selfCollide>
+    <selfCollide>true</selfCollide>
   </gazebo>
   <gazebo reference="l_ank_roll_link">
@@ -59,5 +59,5 @@
     <mu2>0.2</mu2>
     <material>Gazebo/White</material>
-    <selfCollide>false</selfCollide>
+    <selfCollide>true</selfCollide>
   </gazebo>
   <gazebo reference="r_hip_roll_link">
@@ -65,5 +65,5 @@
     <mu2>0.2</mu2>
     <material>Gazebo/White</material>
-    <selfCollide>false</selfCollide>
+    <selfCollide>true</selfCollide>
   </gazebo>
   <gazebo reference="r_hip_pitch_link">
@@ -71,5 +71,5 @@
     <mu2>0.2</mu2>
     <material>Gazebo/White</material>
-    <selfCollide>false</selfCollide>
+    <selfCollide>true</selfCollide>
   </gazebo>
   <gazebo reference="r_knee_link">
@@ -77,5 +77,5 @@
     <mu2>0.2</mu2>
     <material>Gazebo/White</material>
-    <selfCollide>false</selfCollide>
+    <selfCollide>true</selfCollide>
   </gazebo>
   <gazebo reference="r_ank_pitch_link">
@@ -83,5 +83,5 @@
     <mu2>0.2</mu2>
     <material>Gazebo/White</material>
-    <selfCollide>false</selfCollide>
+    <selfCollide>true</selfCollide>
   </gazebo>
   <gazebo reference="r_ank_roll_link">
@@ -100,5 +100,5 @@
     <mu2>0.2</mu2>
     <material>Gazebo/White</material>
-    <selfCollide>false</selfCollide>
+    <selfCollide>true</selfCollide>
   </gazebo>
   <gazebo reference="r_sho_roll_link">
@@ -106,5 +106,5 @@
     <mu2>0.2</mu2>
     <material>Gazebo/White</material>
-    <selfCollide>false</selfCollide>
+    <selfCollide>true</selfCollide>
   </gazebo>
   <gazebo reference="r_el_link">
@@ -112,5 +112,5 @@
     <mu2>0.2</mu2>
     <material>Gazebo/White</material>
-    <selfCollide>false</selfCollide>
+    <selfCollide>true</selfCollide>
   </gazebo>
   <gazebo reference="l_sho_pitch_link">
@@ -118,5 +118,5 @@
     <mu2>0.2</mu2>
     <material>Gazebo/White</material>
-    <selfCollide>false</selfCollide>
+    <selfCollide>true</selfCollide>
   </gazebo>
   <gazebo reference="l_sho_roll_link">
@@ -124,5 +124,5 @@
     <mu2>0.2</mu2>
     <material>Gazebo/White</material>
-    <selfCollide>false</selfCollide>
+    <selfCollide>true</selfCollide>
   </gazebo>
   <gazebo reference="l_el_link">
@@ -130,5 +130,5 @@
     <mu2>0.2</mu2>
     <material>Gazebo/White</material>
-    <selfCollide>false</selfCollide>
+    <selfCollide>true</selfCollide>
   </gazebo>
   <gazebo reference="head_pan_link">
@@ -136,5 +136,5 @@
     <mu2>0.2</mu2>
     <material>Gazebo/White</material>
-    <selfCollide>false</selfCollide>
+    <selfCollide>true</selfCollide>
   </gazebo>
   <gazebo reference="head_tilt_link">
@@ -142,5 +142,5 @@
     <mu2>0.2</mu2>
     <material>Gazebo/White</material>
-    <selfCollide>false</selfCollide>
+    <selfCollide>true</selfCollide>
   </gazebo>
 <!--
@@ -265,5 +265,5 @@
     <sensor name="imu_sensor" type="imu">
       <always_on>true</always_on>
-      <update_rate>100</update_rate>
+      <update_rate>200</update_rate>
       <visualize>true</visualize>
       <topic>__default_topic__</topic>
@@ -271,5 +271,5 @@
         <topicName>robotis_op3/imu</topicName>
         <bodyName>body_link</bodyName>
-        <updateRateHZ>10.0</updateRateHZ>
+        <updateRateHZ>0</updateRateHZ>
         <gaussianNoise>0.0</gaussianNoise>
         <xyzOffset>0 0 0</xyzOffset>

File: op3_gym/urdf_simple/robotis_op3.structure.head.xacro (robot description, xacro)
@@ -12,5 +12,5 @@
     <origin xyz="-0.001 0.0 0.1365" rpy="0 0 0" />
     <axis xyz="0 0 1" />
-    <limit effort="1.51" velocity="100" lower="${-pi*0.9}" upper="${pi*0.9}" />
+    <limit effort="4.1" velocity="100" lower="${-pi*0.9}" upper="${pi*0.9}" />
     <dynamics damping="0.1" friction="0.0" />
   </joint>
@@ -34,5 +34,5 @@
     <origin xyz="0.010 0.019 0.0285" rpy="0 0 0" />
     <axis xyz="0 -1 0" />
-    <limit effort="1.51" velocity="100" lower="${-pi*0.9}" upper="${pi*0.9}" />
+    <limit effort="4.1" velocity="100" lower="${-pi*0.9}" upper="${pi*0.9}" />
     <dynamics damping="0.1" friction="0.0" />
   </joint>

File: op3_gym/urdf_simple/robotis_op3.structure.larm.xacro (robot description, xacro)
@@ -12,5 +12,5 @@
     <origin xyz="-0.001 0.06 0.111" rpy="0 0 0" />
     <axis xyz="0 1 0" />
-    <limit effort="1.51" velocity="100" lower="${-pi*0.9}" upper="${pi*0.9}" />
+    <limit effort="4.1" velocity="100" lower="${-pi*0.9}" upper="${pi*0.9}" />
     <dynamics damping="0.1" friction="0.0" />
   </joint>
@@ -34,5 +34,5 @@
     <origin xyz="0.019 0.0285 -0.010" rpy="0 0 0" />
     <axis xyz="-1 0 0" />
-    <limit effort="1.51" velocity="100" lower="${-pi*0.9}" upper="${pi*0.9}" />
+    <limit effort="4.1" velocity="100" lower="${-pi*0.9}" upper="${pi*0.9}" />
     <dynamics damping="0.1" friction="0.0" />
   </joint>
@@ -56,5 +56,5 @@
     <origin xyz="0.0 0.0904 -0.0001" rpy="0 0 0" />
     <axis xyz="1 0 0" />
-    <limit effort="1.51" velocity="100" lower="${-pi*0.9}" upper="${pi*0.9}" />
+    <limit effort="4.1" velocity="100" lower="${-pi*0.9}" upper="${pi*0.9}" />
     <dynamics damping="0.1" friction="0.0" />
   </joint>

File: op3_gym/urdf_simple/robotis_op3.structure.lleg.xacro (robot description, xacro)
@@ -12,5 +12,5 @@
     <origin xyz="0.0 0.035 0.0" rpy="0 0 0" />
     <axis xyz="0 0 -1" />
-    <limit effort="1.51" velocity="100" lower="${-pi*0.9}" upper="${pi*0.9}" />
+    <limit effort="4.1" velocity="100" lower="${-pi*0.9}" upper="${pi*0.9}" />
     <dynamics damping="0.1" friction="0.0" />
   </joint>
@@ -34,5 +34,5 @@
     <origin xyz="-0.024 0.0 -0.0285" rpy="0 0 0" />
     <axis xyz="-1 0 0" />
-    <limit effort="1.51" velocity="100" lower="${-pi*0.9}" upper="${pi*0.9}" />
+    <limit effort="4.1" velocity="100" lower="${-pi*0.9}" upper="${pi*0.9}" />
     <dynamics damping="0.1" friction="0.0" />
   </joint>
@@ -56,5 +56,5 @@
     <origin xyz="0.0241 0.019 0.0" rpy="0 0 0" />
     <axis xyz="0 1 0" />
-    <limit effort="1.51" velocity="100" lower="${-pi*0.9}" upper="${pi*0.9}" />
+    <limit effort="4.1" velocity="100" lower="${-pi*0.9}" upper="${pi*0.9}" />
     <dynamics damping="0.1" friction="0.0" />
   </joint>
@@ -82,5 +82,5 @@
     <origin xyz="0.0 0.0 -0.11015" rpy="0 0 0" />
     <axis xyz="0 1 0" />
-    <limit effort="1.51" velocity="100" lower="${-pi*0.9}" upper="${pi*0.9}" />
+    <limit effort="4.1" velocity="100" lower="${-pi*0.9}" upper="${pi*0.9}" />
     <dynamics damping="0.1" friction="0.0" />
   </joint>
@@ -108,5 +108,5 @@
     <origin xyz="0 0 -0.110" rpy="0 0 0" />
     <axis xyz="0 -1 0" />
-    <limit effort="1.51" velocity="100" lower="${-pi*0.9}" upper="${pi*0.9}" />
+    <limit effort="4.1" velocity="100" lower="${-pi*0.9}" upper="${pi*0.9}" />
     <dynamics damping="0.1" friction="0.0" />
   </joint>
@@ -130,5 +130,5 @@
     <origin xyz="-0.0241 -0.019 0" rpy="0 0 0" />
     <axis xyz="1 0 0" />
-    <limit effort="1.51" velocity="100" lower="${-pi*0.9}" upper="${pi*0.9}" />
+    <limit effort="4.1" velocity="100" lower="${-pi*0.9}" upper="${pi*0.9}" />
     <dynamics damping="0.1" friction="0.0" />
   </joint>
@@ -145,4 +145,12 @@
         <box size="0.14 0.085 0.01" />
       </geometry>
+      <surface>
+        <friction>
+          <ode>
+            <mu>0.9</mu>
+            <mu2>0.8</mu2>
+          </ode>
+        </friction>
+      </surface>
     </collision>
     <inertial>

File: op3_gym/urdf_simple/robotis_op3.structure.rarm.xacro (robot description, xacro)
@@ -12,5 +12,5 @@
     <origin xyz="-0.001 -0.06 0.111" rpy="0 0 0" />
     <axis xyz="0 -1 0" />
-    <limit effort="1.51" velocity="100" lower="${-pi*0.9}" upper="${pi*0.9}" />
+    <limit effort="4.1" velocity="100" lower="${-pi*0.9}" upper="${pi*0.9}" />
     <dynamics damping="0.1" friction="0.0" />
   </joint>
@@ -34,5 +34,5 @@
     <origin xyz="0.019 -0.0285 -0.010" rpy="0 0 0" />
     <axis xyz="-1 0 0" />
-    <limit effort="1.51" velocity="100" lower="${-pi*0.9}" upper="${pi*0.9}" />
+    <limit effort="4.1" velocity="100" lower="${-pi*0.9}" upper="${pi*0.9}" />
     <dynamics damping="0.1" friction="0.0" />
   </joint>
@@ -56,5 +56,5 @@
     <origin xyz="0.0 -0.0904 -0.0001" rpy="0 0 0" />
     <axis xyz="1 0 0" />
-    <limit effort="1.51" velocity="100" lower="${-pi*0.9}" upper="${pi*0.9}" />
+    <limit effort="4.1" velocity="100" lower="${-pi*0.9}" upper="${pi*0.9}" />
     <dynamics damping="0.1" friction="0.0" />
   </joint>

File: op3_gym/urdf_simple/robotis_op3.structure.rleg.xacro (robot description, xacro)
@@ -12,5 +12,5 @@
     <origin xyz="0.0 -0.035 0.0" rpy="0 0 0" />
     <axis xyz="0 0 -1" />
-    <limit effort="1.51" velocity="100" lower="${-pi*0.9}" upper="${pi*0.9}" />
+    <limit effort="4.1" velocity="100" lower="${-pi*0.9}" upper="${pi*0.9}" />
     <dynamics damping="0.1" friction="0.0" />
   </joint>
@@ -34,5 +34,5 @@
     <origin xyz="-0.024 0.0 -0.0285" rpy="0 0 0" />
     <axis xyz="-1 0 0" />
-    <limit effort="1.51" velocity="100" lower="${-pi*0.9}" upper="${pi*0.9}" />
+    <limit effort="4.1" velocity="100" lower="${-pi*0.9}" upper="${pi*0.9}" />
     <dynamics damping="0.1" friction="0.0" />
   </joint>
@@ -56,5 +56,5 @@
     <origin xyz="0.0241 -0.019 0.0" rpy="0 0 0" />
     <axis xyz="0 -1 0" />
-    <limit effort="1.51" velocity="100" lower="${-pi*0.9}" upper="${pi*0.9}" />
+    <limit effort="4.1" velocity="100" lower="${-pi*0.9}" upper="${pi*0.9}" />
     <dynamics damping="0.1" friction="0.0" />
   </joint>
@@ -82,5 +82,5 @@
     <origin xyz="0.0 0.0 -0.11015" rpy="0 0 0" />
     <axis xyz="0 -1 0" />
-    <limit effort="1.51" velocity="100" lower="${-pi*0.9}" upper="${pi*0.9}" />
+    <limit effort="4.1" velocity="100" lower="${-pi*0.9}" upper="${pi*0.9}" />
     <dynamics damping="0.1" friction="0.0" />
   </joint>
@@ -108,5 +108,5 @@
     <origin xyz="0 0 -0.110" rpy="0 0 0" />
     <axis xyz="0 1 0" />
-    <limit effort="1.51" velocity="100" lower="${-pi*0.9}" upper="${pi*0.9}" />
+    <limit effort="4.1" velocity="100" lower="${-pi*0.9}" upper="${pi*0.9}" />
     <dynamics damping="0.1" friction="0.0" />
   </joint>
@@ -130,5 +130,5 @@
     <origin xyz="-0.0241 0.019 0" rpy="0 0 0" />
     <axis xyz="1 0 0" />
-    <limit effort="1.51" velocity="100" lower="${-pi*0.9}" upper="${pi*0.9}" />
+    <limit effort="4.1" velocity="100" lower="${-pi*0.9}" upper="${pi*0.9}" />
     <dynamics damping="0.1" friction="0.0" />
   </joint>
@@ -145,4 +145,12 @@
         <box size="0.14 0.085 0.01" />
       </geometry>
+      <surface>
+        <friction>
+          <ode>
+            <mu>0.9</mu>
+            <mu2>0.8</mu2>
+          </ode>
+        </friction>
+      </surface>
     </collision>
     <inertial>

File: op3_gym/urdf_simple/robotis_op3.urdf.xacro (robot description, xacro)
@@ -38,7 +38,11 @@
       <xacro:insert_mesh_body_link />
     </visual>
-    <!-- <collision>
-      <xacro:insert_mesh_body_link />
-    </collision> -->
+    <collision>
+      <!-- <xacro:insert_mesh_body_link /> -->
+      <origin xyz="0 0 0.07" rpy="0.0 0.0 0.0"/>
+      <geometry>
+        <box size="0.1 0.1 0.1"/>
+      </geometry>
+    </collision>
     <inertial>
       <xacro:insert_inertia_body_link />
