Commit message: checkpoint 210523

File: op3_gym/urdf/robotis_op3.structure.head.xacro (robot description, xacro)
@@ -12,5 +12,5 @@
     <origin xyz="-0.001 0.0 0.1365" rpy="0 0 0" />
     <axis xyz="0 0 1" />
-    <limit effort="5" velocity="5" lower="${-pi*0.9}" upper="${pi*0.9}" />
+    <limit effort="10" velocity="10" lower="${-pi*0.9}" upper="${pi*0.9}" />
     <dynamics damping="0.1" friction="0.0" />
   </joint>
@@ -34,5 +34,5 @@
     <origin xyz="0.010 0.019 0.0285" rpy="0 0 0" />
     <axis xyz="0 -1 0" />
-    <limit effort="5" velocity="5" lower="${-pi*0.9}" upper="${pi*0.9}" />
+    <limit effort="10" velocity="10" lower="${-pi*0.9}" upper="${pi*0.9}" />
     <dynamics damping="0.1" friction="0.0" />
   </joint>

File: op3_gym/urdf/robotis_op3.structure.larm.xacro (robot description, xacro)
@@ -12,5 +12,5 @@
     <origin xyz="-0.001 0.06 0.111" rpy="0 0 0" />
     <axis xyz="0 1 0" />
-    <limit effort="5" velocity="5" lower="${-pi*0.9}" upper="${pi*0.9}" />
+    <limit effort="10" velocity="10" lower="${-pi*0.9}" upper="${pi*0.9}" />
     <dynamics damping="0.1" friction="0.01" />
   </joint>
@@ -34,5 +34,5 @@
     <origin xyz="0.019 0.0285 -0.010" rpy="0 0 0" />
     <axis xyz="-1 0 0" />
-    <limit effort="5" velocity="5" lower="${-pi*0.9}" upper="${pi*0.9}" />
+    <limit effort="10" velocity="10" lower="${-pi*0.9}" upper="${pi*0.9}" />
     <dynamics damping="0.1" friction="0.01" />
   </joint>
@@ -56,5 +56,5 @@
     <origin xyz="0.0 0.0904 -0.0001" rpy="0 0 0" />
     <axis xyz="1 0 0" />
-    <limit effort="5" velocity="5" lower="${-pi*0.9}" upper="${pi*0.9}" />
+    <limit effort="10" velocity="10" lower="${-pi*0.9}" upper="${pi*0.9}" />
     <dynamics damping="0.1" friction="0.01" />
   </joint>

File: op3_gym/urdf/robotis_op3.structure.lleg.xacro (robot description, xacro)
@@ -12,5 +12,5 @@
     <origin xyz="0.0 0.035 0.0" rpy="0 0 0" />
     <axis xyz="0 0 -1" />
-    <limit effort="5" velocity="5" lower="${-pi*0.9}" upper="${pi*0.9}" />
+    <limit effort="10" velocity="10" lower="${-pi*0.9}" upper="${pi*0.9}" />
     <dynamics damping="0.1" friction="0.0" />
   </joint>
@@ -34,5 +34,5 @@
     <origin xyz="-0.024 0.0 -0.0285" rpy="0 0 0" />
     <axis xyz="-1 0 0" />
-    <limit effort="5" velocity="5" lower="${-pi*0.9}" upper="${pi*0.9}" />
+    <limit effort="10" velocity="10" lower="${-pi*0.9}" upper="${pi*0.9}" />
     <dynamics damping="0.1" friction="0.0" />
   </joint>
@@ -56,5 +56,5 @@
     <origin xyz="0.0241 0.019 0.0" rpy="0 0 0" />
     <axis xyz="0 1 0" />
-    <limit effort="5" velocity="5" lower="${-pi*0.9}" upper="${pi*0.9}" />
+    <limit effort="10" velocity="10" lower="${-pi*0.9}" upper="${pi*0.9}" />
     <dynamics damping="0.1" friction="0.0" />
   </joint>
@@ -78,5 +78,5 @@
     <origin xyz="0.0 0.0 -0.11015" rpy="0 0 0" />
     <axis xyz="0 1 0" />
-    <limit effort="5" velocity="5" lower="${-pi*0.9}" upper="${pi*0.9}" />
+    <limit effort="10" velocity="10" lower="${-pi*0.9}" upper="${pi*0.9}" />
     <dynamics damping="0.1" friction="0.0" />
   </joint>
@@ -100,5 +100,5 @@
     <origin xyz="0 0 -0.110" rpy="0 0 0" />
     <axis xyz="0 -1 0" />
-    <limit effort="5" velocity="5" lower="${-pi*0.9}" upper="${pi*0.9}" />
+    <limit effort="10" velocity="10" lower="${-pi*0.9}" upper="${pi*0.9}" />
     <dynamics damping="0.1" friction="0.0" />
   </joint>
@@ -122,5 +122,5 @@
     <origin xyz="-0.0241 -0.019 0" rpy="0 0 0" />
     <axis xyz="1 0 0" />
-    <limit effort="5" velocity="5" lower="${-pi*0.9}" upper="${pi*0.9}" />
+    <limit effort="10" velocity="10" lower="${-pi*0.9}" upper="${pi*0.9}" />
     <dynamics damping="0.1" friction="0.0" />
   </joint>

File: op3_gym/urdf/robotis_op3.structure.rarm.xacro (robot description, xacro)
@@ -12,5 +12,5 @@
     <origin xyz="-0.001 -0.06 0.111" rpy="0 0 0" />
     <axis xyz="0 -1 0" />
-    <limit effort="5" velocity="5" lower="${-pi*0.9}" upper="${pi*0.9}" />
+    <limit effort="10" velocity="10" lower="${-pi*0.9}" upper="${pi*0.9}" />
     <dynamics damping="0.1" friction="0.0" />
   </joint>
@@ -34,5 +34,5 @@
     <origin xyz="0.019 -0.0285 -0.010" rpy="0 0 0" />
     <axis xyz="-1 0 0" />
-    <limit effort="5" velocity="5" lower="${-pi*0.9}" upper="${pi*0.9}" />
+    <limit effort="10" velocity="10" lower="${-pi*0.9}" upper="${pi*0.9}" />
     <dynamics damping="0.1" friction="0.0" />
   </joint>
@@ -56,5 +56,5 @@
     <origin xyz="0.0 -0.0904 -0.0001" rpy="0 0 0" />
     <axis xyz="1 0 0" />
-    <limit effort="5" velocity="5" lower="${-pi*0.9}" upper="${pi*0.9}" />
+    <limit effort="10" velocity="10" lower="${-pi*0.9}" upper="${pi*0.9}" />
     <dynamics damping="0.1" friction="0.0" />
   </joint>

File: op3_gym/urdf/robotis_op3.structure.rleg.xacro (robot description, xacro)
@@ -12,5 +12,5 @@
     <origin xyz="0.0 -0.035 0.0" rpy="0 0 0" />
     <axis xyz="0 0 -1" />
-    <limit effort="5" velocity="5" lower="${-pi*0.9}" upper="${pi*0.9}" />
+    <limit effort="10" velocity="10" lower="${-pi*0.9}" upper="${pi*0.9}" />
     <dynamics damping="0.1" friction="0.0" />
   </joint>
@@ -34,5 +34,5 @@
     <origin xyz="-0.024 0.0 -0.0285" rpy="0 0 0" />
     <axis xyz="-1 0 0" />
-    <limit effort="5" velocity="5" lower="${-pi*0.9}" upper="${pi*0.9}" />
+    <limit effort="10" velocity="10" lower="${-pi*0.9}" upper="${pi*0.9}" />
     <dynamics damping="0.1" friction="0.0" />
   </joint>
@@ -56,5 +56,5 @@
     <origin xyz="0.0241 -0.019 0.0" rpy="0 0 0" />
     <axis xyz="0 -1 0" />
-    <limit effort="5" velocity="5" lower="${-pi*0.9}" upper="${pi*0.9}" />
+    <limit effort="10" velocity="10" lower="${-pi*0.9}" upper="${pi*0.9}" />
     <dynamics damping="0.1" friction="0.0" />
   </joint>
@@ -78,5 +78,5 @@
     <origin xyz="0.0 0.0 -0.11015" rpy="0 0 0" />
     <axis xyz="0 -1 0" />
-    <limit effort="5" velocity="5" lower="${-pi*0.9}" upper="${pi*0.9}" />
+    <limit effort="10" velocity="10" lower="${-pi*0.9}" upper="${pi*0.9}" />
     <dynamics damping="0.1" friction="0.0" />
   </joint>
@@ -100,5 +100,5 @@
     <origin xyz="0 0 -0.110" rpy="0 0 0" />
     <axis xyz="0 1 0" />
-    <limit effort="5" velocity="5" lower="${-pi*0.9}" upper="${pi*0.9}" />
+    <limit effort="10" velocity="10" lower="${-pi*0.9}" upper="${pi*0.9}" />
     <dynamics damping="0.1" friction="0.0" />
   </joint>
@@ -122,5 +122,5 @@
     <origin xyz="-0.0241 0.019 0" rpy="0 0 0" />
     <axis xyz="1 0 0" />
-    <limit effort="5" velocity="5" lower="${-pi*0.9}" upper="${pi*0.9}" />
+    <limit effort="10" velocity="10" lower="${-pi*0.9}" upper="${pi*0.9}" />
     <dynamics damping="0.1" friction="0.0" />
   </joint>

File: op3_gym/urdf/robotis_op3.urdf (robot description, URDF)
Before this commit: robot robotis_op3, 23 links, 22 joints
Joints:
- joint head_pan: limit lower=-2.827433388230814 upper=2.827433388230814 effort=5 velocity=5 -> lower=-2.827433388230814 upper=2.827433388230814 effort=10 velocity=10
- joint head_tilt: limit lower=-2.827433388230814 upper=2.827433388230814 effort=5 velocity=5 -> lower=-2.827433388230814 upper=2.827433388230814 effort=10 velocity=10
- joint l_ank_pitch: limit lower=-2.827433388230814 upper=2.827433388230814 effort=5 velocity=5 -> lower=-2.827433388230814 upper=2.827433388230814 effort=10 velocity=10
- joint l_ank_roll: limit lower=-2.827433388230814 upper=2.827433388230814 effort=5 velocity=5 -> lower=-2.827433388230814 upper=2.827433388230814 effort=10 velocity=10
- joint l_el: limit lower=-2.827433388230814 upper=2.827433388230814 effort=5 velocity=5 -> lower=-2.827433388230814 upper=2.827433388230814 effort=10 velocity=10
- joint l_hip_pitch: limit lower=-2.827433388230814 upper=2.827433388230814 effort=5 velocity=5 -> lower=-2.827433388230814 upper=2.827433388230814 effort=10 velocity=10
- joint l_hip_roll: limit lower=-2.827433388230814 upper=2.827433388230814 effort=5 velocity=5 -> lower=-2.827433388230814 upper=2.827433388230814 effort=10 velocity=10
- joint l_hip_yaw: limit lower=-2.827433388230814 upper=2.827433388230814 effort=5 velocity=5 -> lower=-2.827433388230814 upper=2.827433388230814 effort=10 velocity=10
- joint l_knee: limit lower=-2.827433388230814 upper=2.827433388230814 effort=5 velocity=5 -> lower=-2.827433388230814 upper=2.827433388230814 effort=10 velocity=10
- joint l_sho_pitch: limit lower=-2.827433388230814 upper=2.827433388230814 effort=5 velocity=5 -> lower=-2.827433388230814 upper=2.827433388230814 effort=10 velocity=10
- joint l_sho_roll: limit lower=-2.827433388230814 upper=2.827433388230814 effort=5 velocity=5 -> lower=-2.827433388230814 upper=2.827433388230814 effort=10 velocity=10
- joint r_ank_pitch: limit lower=-2.827433388230814 upper=2.827433388230814 effort=5 velocity=5 -> lower=-2.827433388230814 upper=2.827433388230814 effort=10 velocity=10
- joint r_ank_roll: limit lower=-2.827433388230814 upper=2.827433388230814 effort=5 velocity=5 -> lower=-2.827433388230814 upper=2.827433388230814 effort=10 velocity=10
- joint r_el: limit lower=-2.827433388230814 upper=2.827433388230814 effort=5 velocity=5 -> lower=-2.827433388230814 upper=2.827433388230814 effort=10 velocity=10
- joint r_hip_pitch: limit lower=-2.827433388230814 upper=2.827433388230814 effort=5 velocity=5 -> lower=-2.827433388230814 upper=2.827433388230814 effort=10 velocity=10
- joint r_hip_roll: limit lower=-2.827433388230814 upper=2.827433388230814 effort=5 velocity=5 -> lower=-2.827433388230814 upper=2.827433388230814 effort=10 velocity=10
- joint r_hip_yaw: limit lower=-2.827433388230814 upper=2.827433388230814 effort=5 velocity=5 -> lower=-2.827433388230814 upper=2.827433388230814 effort=10 velocity=10
- joint r_knee: limit lower=-2.827433388230814 upper=2.827433388230814 effort=5 velocity=5 -> lower=-2.827433388230814 upper=2.827433388230814 effort=10 velocity=10
- joint r_sho_pitch: limit lower=-2.827433388230814 upper=2.827433388230814 effort=5 velocity=5 -> lower=-2.827433388230814 upper=2.827433388230814 effort=10 velocity=10
- joint r_sho_roll: limit lower=-2.827433388230814 upper=2.827433388230814 effort=5 velocity=5 -> lower=-2.827433388230814 upper=2.827433388230814 effort=10 velocity=10

Commit message: kimyoungjin 210921 configs

File: op3_gym/urdf/robotis_op3.structure.head.xacro (robot description, xacro)
@@ -12,5 +12,5 @@
     <origin xyz="-0.001 0.0 0.1365" rpy="0 0 0" />
     <axis xyz="0 0 1" />
-    <limit effort="1.5" velocity="100" lower="${-pi*0.9}" upper="${pi*0.9}" />
+    <limit effort="2.5" velocity="100" lower="${-pi*0.9}" upper="${pi*0.9}" />
     <dynamics damping="0.1" friction="0.0" />
   </joint>
@@ -34,5 +34,5 @@
     <origin xyz="0.010 0.019 0.0285" rpy="0 0 0" />
     <axis xyz="0 -1 0" />
-    <limit effort="1.5" velocity="100" lower="${-pi*0.9}" upper="${pi*0.9}" />
+    <limit effort="2.5" velocity="100" lower="${-pi*0.9}" upper="${pi*0.9}" />
     <dynamics damping="0.1" friction="0.0" />
   </joint>

File: op3_gym/urdf/robotis_op3.structure.larm.xacro (robot description, xacro)
@@ -12,5 +12,5 @@
     <origin xyz="-0.001 0.06 0.111" rpy="0 0 0" />
     <axis xyz="0 1 0" />
-    <limit effort="1.5" velocity="100" lower="${-pi*0.9}" upper="${pi*0.9}" />
+    <limit effort="2.5" velocity="100" lower="${-pi*0.9}" upper="${pi*0.9}" />
     <dynamics damping="0.1" friction="0.01" />
   </joint>
@@ -34,5 +34,5 @@
     <origin xyz="0.019 0.0285 -0.010" rpy="0 0 0" />
     <axis xyz="-1 0 0" />
-    <limit effort="1.5" velocity="100" lower="${-pi*0.9}" upper="${pi*0.9}" />
+    <limit effort="2.5" velocity="100" lower="${-pi*0.9}" upper="${pi*0.9}" />
     <dynamics damping="0.1" friction="0.01" />
   </joint>
@@ -56,5 +56,5 @@
     <origin xyz="0.0 0.0904 -0.0001" rpy="0 0 0" />
     <axis xyz="1 0 0" />
-    <limit effort="1.5" velocity="100" lower="${-pi*0.9}" upper="${pi*0.9}" />
+    <limit effort="2.5" velocity="100" lower="${-pi*0.9}" upper="${pi*0.9}" />
     <dynamics damping="0.1" friction="0.01" />
   </joint>

File: op3_gym/urdf/robotis_op3.structure.lleg.xacro (robot description, xacro)
@@ -12,5 +12,5 @@
     <origin xyz="0.0 0.035 0.0" rpy="0 0 0" />
     <axis xyz="0 0 -1" />
-    <limit effort="1.5" velocity="100" lower="${-pi*0.9}" upper="${pi*0.9}" />
+    <limit effort="2.5" velocity="100" lower="${-pi*0.9}" upper="${pi*0.9}" />
     <dynamics damping="0.1" friction="0.0" />
   </joint>
@@ -34,5 +34,5 @@
     <origin xyz="-0.024 0.0 -0.0285" rpy="0 0 0" />
     <axis xyz="-1 0 0" />
-    <limit effort="1.5" velocity="100" lower="${-pi*0.9}" upper="${pi*0.9}" />
+    <limit effort="2.5" velocity="100" lower="${-pi*0.9}" upper="${pi*0.9}" />
     <dynamics damping="0.1" friction="0.0" />
   </joint>
@@ -56,5 +56,5 @@
     <origin xyz="0.0241 0.019 0.0" rpy="0 0 0" />
     <axis xyz="0 1 0" />
-    <limit effort="1.5" velocity="100" lower="${-pi*0.9}" upper="${pi*0.9}" />
+    <limit effort="2.5" velocity="100" lower="${-pi*0.9}" upper="${pi*0.9}" />
     <dynamics damping="0.1" friction="0.0" />
   </joint>
@@ -78,5 +78,5 @@
     <origin xyz="0.0 0.0 -0.11015" rpy="0 0 0" />
     <axis xyz="0 1 0" />
-    <limit effort="1.5" velocity="100" lower="${-pi*0.9}" upper="${pi*0.9}" />
+    <limit effort="2.5" velocity="100" lower="${-pi*0.9}" upper="${pi*0.9}" />
     <dynamics damping="0.1" friction="0.0" />
   </joint>
@@ -100,5 +100,5 @@
     <origin xyz="0 0 -0.110" rpy="0 0 0" />
     <axis xyz="0 -1 0" />
-    <limit effort="1.5" velocity="100" lower="${-pi*0.9}" upper="${pi*0.9}" />
+    <limit effort="2.5" velocity="100" lower="${-pi*0.9}" upper="${pi*0.9}" />
     <dynamics damping="0.1" friction="0.0" />
   </joint>
@@ -122,5 +122,5 @@
     <origin xyz="-0.0241 -0.019 0" rpy="0 0 0" />
     <axis xyz="1 0 0" />
-    <limit effort="1.5" velocity="100" lower="${-pi*0.9}" upper="${pi*0.9}" />
+    <limit effort="2.5" velocity="100" lower="${-pi*0.9}" upper="${pi*0.9}" />
     <dynamics damping="0.1" friction="0.0" />
   </joint>

File: op3_gym/urdf/robotis_op3.structure.rarm.xacro (robot description, xacro)
@@ -12,5 +12,5 @@
     <origin xyz="-0.001 -0.06 0.111" rpy="0 0 0" />
     <axis xyz="0 -1 0" />
-    <limit effort="1.5" velocity="100" lower="${-pi*0.9}" upper="${pi*0.9}" />
+    <limit effort="2.5" velocity="100" lower="${-pi*0.9}" upper="${pi*0.9}" />
     <dynamics damping="0.1" friction="0.0" />
   </joint>
@@ -34,5 +34,5 @@
     <origin xyz="0.019 -0.0285 -0.010" rpy="0 0 0" />
     <axis xyz="-1 0 0" />
-    <limit effort="1.5" velocity="100" lower="${-pi*0.9}" upper="${pi*0.9}" />
+    <limit effort="2.5" velocity="100" lower="${-pi*0.9}" upper="${pi*0.9}" />
     <dynamics damping="0.1" friction="0.0" />
   </joint>
@@ -56,5 +56,5 @@
     <origin xyz="0.0 -0.0904 -0.0001" rpy="0 0 0" />
     <axis xyz="1 0 0" />
-    <limit effort="1.5" velocity="100" lower="${-pi*0.9}" upper="${pi*0.9}" />
+    <limit effort="2.5" velocity="100" lower="${-pi*0.9}" upper="${pi*0.9}" />
     <dynamics damping="0.1" friction="0.0" />
   </joint>

File: op3_gym/urdf/robotis_op3.structure.rleg.xacro (robot description, xacro)
@@ -12,5 +12,5 @@
     <origin xyz="0.0 -0.035 0.0" rpy="0 0 0" />
     <axis xyz="0 0 -1" />
-    <limit effort="1.5" velocity="100" lower="${-pi*0.9}" upper="${pi*0.9}" />
+    <limit effort="2.5" velocity="100" lower="${-pi*0.9}" upper="${pi*0.9}" />
     <dynamics damping="0.1" friction="0.0" />
   </joint>
@@ -34,5 +34,5 @@
     <origin xyz="-0.024 0.0 -0.0285" rpy="0 0 0" />
     <axis xyz="-1 0 0" />
-    <limit effort="1.5" velocity="100" lower="${-pi*0.9}" upper="${pi*0.9}" />
+    <limit effort="2.5" velocity="100" lower="${-pi*0.9}" upper="${pi*0.9}" />
     <dynamics damping="0.1" friction="0.0" />
   </joint>
@@ -56,5 +56,5 @@
     <origin xyz="0.0241 -0.019 0.0" rpy="0 0 0" />
     <axis xyz="0 -1 0" />
-    <limit effort="1.5" velocity="100" lower="${-pi*0.9}" upper="${pi*0.9}" />
+    <limit effort="2.5" velocity="100" lower="${-pi*0.9}" upper="${pi*0.9}" />
     <dynamics damping="0.1" friction="0.0" />
   </joint>
@@ -78,5 +78,5 @@
     <origin xyz="0.0 0.0 -0.11015" rpy="0 0 0" />
     <axis xyz="0 -1 0" />
-    <limit effort="1.5" velocity="100" lower="${-pi*0.9}" upper="${pi*0.9}" />
+    <limit effort="2.5" velocity="100" lower="${-pi*0.9}" upper="${pi*0.9}" />
     <dynamics damping="0.1" friction="0.0" />
   </joint>
@@ -100,5 +100,5 @@
     <origin xyz="0 0 -0.110" rpy="0 0 0" />
     <axis xyz="0 1 0" />
-    <limit effort="1.5" velocity="100" lower="${-pi*0.9}" upper="${pi*0.9}" />
+    <limit effort="2.5" velocity="100" lower="${-pi*0.9}" upper="${pi*0.9}" />
     <dynamics damping="0.1" friction="0.0" />
   </joint>
@@ -122,5 +122,5 @@
     <origin xyz="-0.0241 0.019 0" rpy="0 0 0" />
     <axis xyz="1 0 0" />
-    <limit effort="1.5" velocity="100" lower="${-pi*0.9}" upper="${pi*0.9}" />
+    <limit effort="2.5" velocity="100" lower="${-pi*0.9}" upper="${pi*0.9}" />
     <dynamics damping="0.1" friction="0.0" />
   </joint>
